File: Atari 130XE.sch (KiCad schematic (older format))
At the start: 0 parts

Commit message: Memory and Freddie
Changed lines of the file:
@@
 $Descr A4 11693 8268
 encoding utf-8
-Sheet 1 3
+Sheet 1 13
 Title ""
 Date ""
@@
 $EndSheet
 $Sheet
-S 2450 1125 1200 1175
+S 2650 1125 1225 1175
 U 6016CC42
 F0 "Power" 50
 F1 "Power.sch" 50
 $EndSheet
+$Sheet
+S 1050 2800 1225 1175
+U 6019B50C
+F0 "Video" 50
+F1 "Video.sch" 50
+$EndSheet
+$Sheet
+S 4250 1125 1225 1175
+U 601DB005
+F0 "Freddie" 50
+F1 "Freddie.sch" 50
+$EndSheet
+$Sheet
+S 5850 1125 1225 1175
+U 601DB1AF
+F0 "Memory" 50
+F1 "Memory.sch" 50
+$EndSheet
+$Sheet
+S 2650 2800 1225 1175
+U 6022EB24
+F0 "Cartridge" 50
+F1 "Cartridge.sch" 50
+$EndSheet
+$Sheet
+S 7500 1125 1225 1200
+U 60205A08
+F0 "Sally and Antic" 50
+F1 "Sally_Antic.sch" 50
+$EndSheet
+$Sheet
+S 9175 1125 1225 1200
+U 60205B84
+F0 "GTIA" 50
+F1 "GTIA.sch" 50
+$EndSheet
+$Sheet
+S 4250 2800 1225 1175
+U 60205D27
+F0 "PIA" 50
+F1 "PIA.sch" 50
+$EndSheet
+$Sheet
+S 5850 2800 1225 1175
+U 60205DA4
+F0 "POKEY" 50
+F1 "POKEY.sch" 50
+$EndSheet
+$Sheet
+S 7500 2800 1225 1175
+U 60205E1E
+F0 "OSS" 50
+F1 "OSS.sch" 50
+$EndSheet
+$Sheet
+S 9175 2800 1225 1175
+U 60205EE8
+F0 "BASIC" 50
+F1 "BASIC.sch" 50
+$EndSheet
 $EndSCHEMATC

Commit message: GTIA
Changed lines of the file:
@@
 $Descr A4 11693 8268
 encoding utf-8
-Sheet 1 13
+Sheet 1 14
 Title ""
 Date ""
@@
 F1 "BASIC.sch" 50
 $EndSheet
+$Sheet
+S 1050 4475 1225 1175
+U 60250803
+F0 "MMU" 50
+F1 "MMU.sch" 50
+$EndSheet
 $EndSCHEMATC

Commit message: MMU, Joy, Cart and Video
Changed lines of the file:
@@
 $Descr A4 11693 8268
 encoding utf-8
-Sheet 1 14
+Sheet 1 15
 Title ""
 Date ""
@@
 S 1050 2800 1225 1175
 U 6019B50C
-F0 "Video" 50
-F1 "Video.sch" 50
+F0 "Audio and Video" 50
+F1 "Audio and Video.sch" 50
 $EndSheet
 $Sheet
@@
 F1 "MMU.sch" 50
 $EndSheet
+$Sheet
+S 2650 4475 1225 1175
+U 602D08E2
+F0 "Ports" 50
+F1 "Ports.sch" 50
+$EndSheet
 $EndSCHEMATC
