File: Atari 130XE.kicad_pcb (KiCad board)
At the start: 2 copper layers, 324 x 204 mm, 24 parts, among them J7 Power, SW1 Switch_power_on

Commit message: Memory and Freddie
Parts:
- added C1: 470uF, Capacitor_THT:CP_Radial_D8.0mm_P3.80mm, F.Cu at (6.81, 35.5)
- added C10: 22uF, Capacitor_THT:CP_Radial_D6.3mm_P2.50mm, F.Cu at (41.7, 36.3)
- added C103: 100nF, Atari:C_Axial_L5.1mm_D2.5mm_P12.50mm_Horizontal, F.Cu at (62.7, 141.0)
- added C11: 10nF, Atari:C_Axial_L5.1mm_D2.5mm_P12.50mm_Horizontal, F.Cu at (32.1, 54.9)
- added C12: 1nF, Atari:C_Axial_L5.1mm_D2.5mm_P12.50mm_Horizontal, F.Cu at (31.0, 31.0)
- added C13: 100nF, Atari:C_Axial_L5.1mm_D2.5mm_P12.50mm_Horizontal, F.Cu at (48.0, 45.9)
- added C14: 1nF, Atari:C_Axial_L5.1mm_D2.5mm_P12.50mm_Horizontal, F.Cu at (27.8, 31.0)
- added C15: 1nF, Atari:C_Axial_L5.1mm_D2.5mm_P12.50mm_Horizontal, F.Cu at (48.0, 48.8)
- added C2: 22uF, Capacitor_THT:CP_Radial_D6.3mm_P2.50mm, F.Cu at (19.6, 36.3)
- added C205: 100nF, Atari:C_Axial_L5.1mm_D2.5mm_P12.50mm_Horizontal, F.Cu at (98.3, 78.0)
- added C27: 100nF, Atari:C_Axial_L5.1mm_D2.5mm_P12.50mm_Horizontal, F.Cu at (152.0, 142.0)
- added C28: 100nF, Atari:C_Axial_L5.1mm_D2.5mm_P12.50mm_Horizontal, F.Cu at (152.0, 139.0)
- added C29: 100nF, Atari:C_Axial_L5.1mm_D2.5mm_P12.50mm_Horizontal, F.Cu at (22.8, 160.8)
- added C3: 22uF, Capacitor_THT:CP_Radial_D6.3mm_P2.50mm, F.Cu at (46.5, 7.18)
- added C32: 100nF, Atari:C_Axial_L5.1mm_D2.5mm_P12.50mm_Horizontal, F.Cu at (44.7, 187.0)
- added C33: 100nF, Atari:C_Axial_L5.1mm_D2.5mm_P12.50mm_Horizontal, F.Cu at (44.7, 189.7)
- added C34: 100nF, Capacitor_THT:C_Axial_L3.8mm_D2.6mm_P7.50mm_Horizontal, F.Cu at (14.4, 106.6)
- added C35: 100nF, Capacitor_THT:C_Axial_L3.8mm_D2.6mm_P7.50mm_Horizontal, F.Cu at (14.4, 68.5)
- added C36: 100nF, Capacitor_THT:C_Axial_L3.8mm_D2.6mm_P7.50mm_Horizontal, F.Cu at (14.4, 81.2)
- added C37: 100nF, Capacitor_THT:C_Axial_L3.8mm_D2.6mm_P7.50mm_Horizontal, F.Cu at (14.4, 93.9)
- added C4: 100nF, Atari:C_Axial_L5.1mm_D2.5mm_P12.50mm_Horizontal, F.Cu at (19.6, 42.5)
- added C5: 1nF, Atari:C_Axial_L5.1mm_D2.5mm_P12.50mm_Horizontal, F.Cu at (19.6, 45.5)
- added C6: 1nF, Atari:C_Axial_L5.1mm_D2.5mm_P12.50mm_Horizontal, F.Cu at (15.3, 22.7)
- added C7: 10nF, Atari:C_Axial_L5.1mm_D2.5mm_P12.50mm_Horizontal, F.Cu at (15.3, 28.2)
- added C8: 1nF, Atari:C_Axial_L5.1mm_D2.5mm_P12.50mm_Horizontal, F.Cu at (32.1, 51.9)
- added C9: 1nF, Atari:C_Axial_L5.1mm_D2.5mm_P12.50mm_Horizontal, F.Cu at (31.0, 28.2)
- added FB1: Ferrite_Bead, Atari:L_Axial_L7.0mm_D3.3mm_P12.50mm_Horizontal_Fastron_MICC, F.Cu at (32.1, 48.7)
- added FB103: Ferrite_Bead, Atari:L_Axial_L7.0mm_D3.3mm_P12.50mm_Horizontal_Fastron_MICC, F.Cu at (26.1, 173.3)
- added FB2: Ferrite_Bead, Atari:L_Axial_L7.0mm_D3.3mm_P12.50mm_Horizontal_Fastron_MICC, F.Cu at (43.5, 22.8)
- added FB3: Ferrite_Bead, Atari:L_Axial_L7.0mm_D3.3mm_P12.50mm_Horizontal_Fastron_MICC, F.Cu at (48.0, 42.5)
- added J100: cond, Connector_PinHeader_2.00mm:PinHeader_1x01_P2.00mm_Vertical, F.Cu at (49.7, 187.0)
- added J101: cond, Connector_PinHeader_2.00mm:PinHeader_1x01_P2.00mm_Vertical, F.Cu at (49.7, 189.7)
- added J2: DIN-5_180degree, Atari:DIN_5_pin, F.Cu at (102.3, 12.6)
- added J4: Expansion, Atari:Expansion_Slot, F.Cu at (141.5, 24.0)
- added L13: 820uH, Atari:L_Axial_L7.0mm_D3.3mm_P12.50mm_Horizontal_Fastron_MICC, F.Cu at (94.6, 78.0)
- added M1: Modulator, Atari:Modulator_TV, F.Cu at (52.5, 28.1)
- added R110: 33, Atari:R_Axial_DIN0207_L3.6mm_D2.2mm_P10.16mm_Horizontal, F.Cu at (63.0, 119.0)
- added R111: 33, Atari:R_Axial_DIN0207_L3.6mm_D2.2mm_P10.16mm_Horizontal, F.Cu at (63.0, 122.0)
- added R18: 240, Atari:R_Axial_DIN0207_L3.6mm_D2.2mm_P10.16mm_Horizontal, F.Cu at (38.7, 179.8)
- added R19: 3k, Atari:R_Axial_DIN0207_L3.6mm_D2.2mm_P10.16mm_Horizontal, F.Cu at (259.0, 113.0)
- added R20: 3k, Atari:R_Axial_DIN0207_L3.6mm_D2.2mm_P10.16mm_Horizontal, F.Cu at (118.0, 38.0)
- added R207: 33, Atari:R_Axial_DIN0207_L3.6mm_D2.2mm_P10.16mm_Horizontal, F.Cu at (44.0, 71.0)
- added R208: 33, Atari:R_Axial_DIN0207_L3.6mm_D2.2mm_P10.16mm_Horizontal, F.Cu at (44.0, 67.0)
- added R209: 33, Atari:R_Axial_DIN0207_L3.6mm_D2.2mm_P10.16mm_Horizontal, F.Cu at (47.0, 82.0)
- added R210: 33, Atari:R_Axial_DIN0207_L3.6mm_D2.2mm_P10.16mm_Horizontal, F.Cu at (47.0, 86.0)
- added R211: 33, Atari:R_Axial_DIN0207_L3.6mm_D2.2mm_P10.16mm_Horizontal, F.Cu at (47.0, 94.0)
- added R212: 33, Atari:R_Axial_DIN0207_L3.6mm_D2.2mm_P10.16mm_Horizontal, F.Cu at (47.0, 90.0)
- added R213: 33, Atari:R_Axial_DIN0207_L3.6mm_D2.2mm_P10.16mm_Horizontal, F.Cu at (44.0, 75.0)
- added R214: 33, Atari:R_Axial_DIN0207_L3.6mm_D2.2mm_P10.16mm_Horizontal, F.Cu at (44.0, 79.0)
- added R26: 1M, Atari:R_Axial_DIN0207_L3.6mm_D2.2mm_P10.16mm_Horizontal, F.Cu at (41.3, 179.8)
- added R30: 3k, Atari:R_Axial_DIN0207_L3.6mm_D2.2mm_P10.16mm_Horizontal, F.Cu at (84.0, 161.0)
- added U10: DRAM_4464, Package_DIP:DIP-18_W7.62mm, F.Cu at (17.5, 81.3)
- added U11: DRAM_4464, Package_DIP:DIP-18_W7.62mm, F.Cu at (17.5, 94.0)
- added U12: DRAM_4464, Package_DIP:DIP-18_W7.62mm, F.Cu at (17.5, 106.7)
- added U18: 74LS08, Package_DIP:DIP-14_W7.62mm_Socket, F.Cu at (239.0, 102.0)
- added U34: MMMU, Package_DIP:DIP-16_W7.62mm_Socket, F.Cu at (61.3, 137.4)
- added U4: BASIC_ROM, Package_DIP:DIP-24_W15.24mm_Socket, F.Cu at (152.0, 161.0)
- added U5: 27C128, Package_DIP:DIP-28_W15.24mm_Socket, F.Cu at (146.9, 134.0)
- added U6: Freddie, Package_DIP:DIP-40_W15.24mm_Socket, F.Cu at (30.0, 176.0)
- added U9: DRAM_4464, Package_DIP:DIP-18_W7.62mm, F.Cu at (17.5, 68.6)
- added Y1: Crystal, Crystal:Crystal_HC18-U_Vertical, F.Cu at (34.0, 184.8)
- moved J7 0.45 mm to (32.0, 12.6)
Connections:
- SW1 pad 2: (no net) -> Net-(C1-Pad1)
Routing:
- net +5VA: track 0.00 -> 660.3 mm, vias 0 -> 6
- net GND: track 0.00 -> 261.0 mm, vias 0 -> 2
- net A0: track 0.00 -> 176.0 mm, vias 0 -> 1
- net A1: track 0.00 -> 170.1 mm, vias 0 -> 1
- net A2: track 0.00 -> 164.1 mm, vias 0 -> 1
- net A11: track 0.00 -> 162.7 mm, vias 0 -> 3
- net A3: track 0.00 -> 158.7 mm, vias 0 -> 1
- net A12: track 0.00 -> 158.1 mm, vias 0 -> 3
- net A10: track 0.00 -> 156.2 mm, vias 0 -> 1
- net A4: track 0.00 -> 152.4 mm, vias 0 -> 1
- net A9: track 0.00 -> 151.1 mm, vias 0 -> 1
- net A8: track 0.00 -> 149.8 mm, vias 0 -> 1
- net A5: track 0.00 -> 146.5 mm, vias 0 -> 1
- net A6: track 0.00 -> 140.9 mm, vias 0 -> 1
- net A7: track 0.00 -> 136.4 mm, vias 0 -> 1
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
Commit message: GTIA
Parts:
- added C42: 100nF, Capacitor_THT:C_Axial_L3.8mm_D2.6mm_P7.50mm_Horizontal, F.Cu at (160.9, 107.8)
- added U17: GTIA, Package_DIP:DIP-40_W15.24mm_Socket, F.Cu at (131.7, 103.8)

Commit message: GTIA put on board
Parts:
- added C111: 820pF, Atari:C_Axial_L5.1mm_D2.5mm_P12.50mm_Horizontal, F.Cu at (89.9, 147.5)
- added C206: 22pF, Atari:C_Axial_L5.1mm_D2.5mm_P12.50mm_Horizontal, F.Cu at (143.0, 151.5)
- added C30: 100nF, Atari:C_Axial_L5.1mm_D2.5mm_P12.50mm_Horizontal, F.Cu at (131.7, 89.0)
- added C31: 100nF, Atari:C_Axial_L5.1mm_D2.5mm_P12.50mm_Horizontal, F.Cu at (131.7, 63.0)
- added C44: 68pF, Atari:C_Axial_L5.1mm_D2.5mm_P12.50mm_Horizontal, F.Cu at (197.7, -54.4)
- added C45: 220pF, Atari:C_Axial_L5.1mm_D2.5mm_P12.50mm_Horizontal, F.Cu at (156.1, -16.4)
- added C46: 1nF, Atari:C_Axial_L5.1mm_D2.5mm_P12.50mm_Horizontal, F.Cu at (171.8, -25.4)
- added C47: 1nF, Atari:C_Axial_L5.1mm_D2.5mm_P12.50mm_Horizontal, F.Cu at (182.0, -43.7)
- added C48: 100nF, Atari:C_Axial_L5.1mm_D2.5mm_P12.50mm_Horizontal, F.Cu at (167.9, -28.9)
- added C50: 10uF, Capacitor_THT:CP_Radial_D5.0mm_P2.00mm, F.Cu at (102.2, 102.4)
- added C51: 100nF, Atari:C_Axial_L5.1mm_D2.5mm_P12.50mm_Horizontal, F.Cu at (98.1, 105.0)
- added C58: 100nF, Atari:C_Axial_L5.1mm_D2.5mm_P12.50mm_Horizontal, F.Cu at (130.4, 137.0)
- added C59: 22pF, Atari:C_Axial_L5.1mm_D2.5mm_P12.50mm_Horizontal, F.Cu at (127.2, 151.5)
- added C60: 560pF, Atari:C_Axial_L5.1mm_D2.5mm_P12.50mm_Horizontal, F.Cu at (139.2, 151.5)
- added C61: 100nF, Atari:C_Axial_L5.1mm_D2.5mm_P12.50mm_Horizontal, F.Cu at (89.9, 151.5)
- added C96: 1nF, Atari:C_Axial_L5.1mm_D2.5mm_P12.50mm_Horizontal, F.Cu at (182.0, -50.8)
- added C97: 1nF, Atari:C_Axial_L5.1mm_D2.5mm_P12.50mm_Horizontal, F.Cu at (167.9, -36.0)
- added D2: 1N4148, Diode_THT:D_DO-35_SOD27_P7.62mm_Horizontal, F.Cu at (240.0, -47.2)
- added D3: 1N4148, Diode_THT:D_DO-35_SOD27_P7.62mm_Horizontal, F.Cu at (240.0, -50.8)
- added D4: 1N4148, Diode_THT:D_DO-35_SOD27_P12.70mm_Horizontal, F.Cu at (111.1, 86.4)
- added FB31: Ferrite_Bead, Atari:L_Axial_L7.0mm_D3.3mm_P12.50mm_Horizontal_Fastron_MICC, F.Cu at (91.9, 92.5)
- added FB9: Ferrite_Bead, Atari:L_Axial_L7.0mm_D3.3mm_P12.50mm_Horizontal_Fastron_MICC, F.Cu at (213.3, -57.3)
- added L23: 100uH, Atari:L_Axial_L7.0mm_D3.3mm_P12.50mm_Horizontal_Fastron_MICC, F.Cu at (183.5, -39.5)
- added L30: 100uH, Atari:L_Axial_L7.0mm_D3.3mm_P12.50mm_Horizontal_Fastron_MICC, F.Cu at (197.7, -45.3)
- added L32: 100uH, Atari:L_Axial_L7.0mm_D3.3mm_P12.50mm_Horizontal_Fastron_MICC, F.Cu at (86.9, 102.4)
- added L37: Bead or 470R, Atari:L_Axial_L7.0mm_D3.3mm_P12.50mm_Horizontal_Fastron_MICC, F.Cu at (135.2, 151.5)
- added L5: 820uH, Atari:L_Axial_L7.0mm_D3.3mm_P12.50mm_Horizontal_Fastron_MICC, F.Cu at (94.9, 105.0)
- added L6: 100uH, Atari:L_Axial_L7.0mm_D3.3mm_P12.50mm_Horizontal_Fastron_MICC, F.Cu at (108.5, 114.0)
- added L8: 1,5uH, Atari:L_Axial_L7.0mm_D3.3mm_P12.50mm_Horizontal_Fastron_MICC, F.Cu at (89.9, 143.5)
- added Q1: 2N3904, Package_TO_SOT_THT:TO-92, F.Cu at (242.7, -56.5)
- added Q2: 2N3904, Package_TO_SOT_THT:TO-92, F.Cu at (95.5, 114.2)
- added Q3: 2N3904, Package_TO_SOT_THT:TO-92, F.Cu at (212.1, -9.16)
- added Q6: 2N3904, Package_TO_SOT_THT:TO-92, F.Cu at (124.4, 145.6)
- added R116: 51, Atari:R_Axial_DIN0207_L3.6mm_D2.2mm_P10.16mm_Horizontal, F.Cu at (106.0, 86.4)
- added R132: 220, Atari:R_Axial_DIN0207_L3.6mm_D2.2mm_P10.16mm_Horizontal, F.Cu at (214.7, -27.9)
- added R133: 220, Atari:R_Axial_DIN0207_L3.6mm_D2.2mm_P10.16mm_Horizontal, F.Cu at (226.7, -40.0)
- added R134: 470, Atari:R_Axial_DIN0207_L3.6mm_D2.2mm_P10.16mm_Horizontal, F.Cu at (214.7, -20.8)
- added R135: 470, Atari:R_Axial_DIN0207_L3.6mm_D2.2mm_P10.16mm_Horizontal, F.Cu at (214.1, -16.0)
- added R136: 470, Atari:R_Axial_DIN0207_L3.6mm_D2.2mm_P10.16mm_Horizontal, F.Cu at (225.8, -32.8)
- added R201: 6k8, Atari:R_Axial_DIN0207_L3.6mm_D2.2mm_P10.16mm_Horizontal, F.Cu at (87.1, 118.6)
- added R202: 180, Atari:R_Axial_DIN0207_L3.6mm_D2.2mm_P10.16mm_Horizontal, F.Cu at (90.1, 110.5)
- added R203: 3k3, Atari:R_Axial_DIN0207_L3.6mm_D2.2mm_P10.16mm_Horizontal, F.Cu at (111.1, 114.0)
- added R204: 47, Atari:R_Axial_DIN0207_L3.6mm_D2.2mm_P10.16mm_Horizontal, F.Cu at (198.4, -10.6)
- added R205: 150, Atari:R_Axial_DIN0207_L3.6mm_D2.2mm_P10.16mm_Horizontal, F.Cu at (90.1, 107.6)
- added R31: 3k, Atari:R_Axial_DIN0207_L3.6mm_D2.2mm_P10.16mm_Horizontal, F.Cu at (171.8, -65.0)
- added R35: 33k, Atari:R_Axial_DIN0207_L3.6mm_D2.2mm_P10.16mm_Horizontal, F.Cu at (199.2, -41.1)
- added R36: 680, Atari:R_Axial_DIN0207_L3.6mm_D2.2mm_P10.16mm_Horizontal, F.Cu at (171.8, -12.1)
- added R37: 1k, Atari:R_Axial_DIN0207_L3.6mm_D2.2mm_P10.16mm_Horizontal, F.Cu at (213.3, -49.5)
- added R41: 1k, Atari:R_Axial_DIN0207_L3.6mm_D2.2mm_P10.16mm_Horizontal, F.Cu at (123.8, 114.0)
- added R42: 1k, Atari:R_Axial_DIN0207_L3.6mm_D2.2mm_P10.16mm_Horizontal, F.Cu at (116.2, 114.0)
- added R43: 1k, Atari:R_Axial_DIN0207_L3.6mm_D2.2mm_P10.16mm_Horizontal, F.Cu at (118.7, 114.0)
- added R44: 1k, Atari:R_Axial_DIN0207_L3.6mm_D2.2mm_P10.16mm_Horizontal, F.Cu at (121.2, 114.0)
- added R45: 1k, Atari:R_Axial_DIN0207_L3.6mm_D2.2mm_P10.16mm_Horizontal, F.Cu at (113.6, 114.0)
- added R46: 1k6, Atari:R_Axial_DIN0207_L3.6mm_D2.2mm_P10.16mm_Horizontal, F.Cu at (108.5, 86.4)
- added R47: 36k, Atari:R_Axial_DIN0207_L3.6mm_D2.2mm_P10.16mm_Horizontal, F.Cu at (121.2, 73.9)
- added R48: 18k, Atari:R_Axial_DIN0207_L3.6mm_D2.2mm_P10.16mm_Horizontal, F.Cu at (118.7, 73.9)
- added R49: 9k1, Atari:R_Axial_DIN0207_L3.6mm_D2.2mm_P10.16mm_Horizontal, F.Cu at (116.2, 73.9)
- added R50: 4k7, Atari:R_Axial_DIN0207_L3.6mm_D2.2mm_P10.16mm_Horizontal, F.Cu at (113.6, 73.9)
- added R51: 750, Atari:R_Axial_DIN0207_L3.6mm_D2.2mm_P10.16mm_Horizontal, F.Cu at (103.5, 73.9)
- added R52: 2k, Atari:R_Axial_DIN0207_L3.6mm_D2.2mm_P10.16mm_Horizontal, F.Cu at (229.0, -57.9)
- added R53: 100, Atari:R_Axial_DIN0207_L3.6mm_D2.2mm_P10.16mm_Horizontal, F.Cu at (199.2, -30.3)
- added R69: 6k8, Atari:R_Axial_DIN0207_L3.6mm_D2.2mm_P10.16mm_Horizontal, F.Cu at (123.2, 164.0)
- added R70: 10k, Atari:R_Axial_DIN0207_L3.6mm_D2.2mm_P10.16mm_Horizontal, F.Cu at (124.5, 137.7)
- added R71: 470, Atari:R_Axial_DIN0207_L3.6mm_D2.2mm_P10.16mm_Horizontal, F.Cu at (102.4, 139.5)
- added R72: 1k, Atari:R_Axial_DIN0207_L3.6mm_D2.2mm_P10.16mm_Horizontal, F.Cu at (112.0, 134.5)
- added R73: 4k7, Atari:R_Axial_DIN0207_L3.6mm_D2.2mm_P10.16mm_Horizontal, F.Cu at (131.2, 151.5)
- added RV38: 500k, Potentiometer_THT:Potentiometer_ACP_CA9-V10_Vertical_Hole, F.Cu at (84.5, 82.0)
- added U20: 4050, Package_DIP:DIP-16_W7.62mm_Socket, F.Cu at (106.0, 98.0)
- added U21: 74LS74, Package_DIP:DIP-14_W7.62mm_Socket, F.Cu at (129.0, 148.0)
- added U7: Antic, Package_DIP:DIP-40_W15.24mm_Socket, F.Cu at (131.7, 84.0)
- added U8: Sally, Package_DIP:DIP-40_W15.24mm_Socket, F.Cu at (131.7, 58.0)
- added Y2: 4,43 MHz, Crystal:Crystal_HC18-U_Horizontal, F.Cu at (132.0, 169.0)
- C42: footprint Capacitor_THT:C_Axial_L3.8mm_D2.6mm_P7.50mm_Horizontal -> Atari:C_Axial_L5.1mm_D2.5mm_P12.50mm_Horizontal
- moved C42 30.1 mm to (131.7, 115.0)
- moved U17 5.18 mm to (131.7, 109.0)
Connections:
- J4 pad 6: (no net) -> REF
- J4 pad B: (no net) -> IRQ
- U17 pad 12: (no net) -> Net-(R134-Pad2)
- U17 pad 13: (no net) -> Net-(R135-Pad2)
- U17 pad 14: (no net) -> Net-(R136-Pad2)
- U17 pad 16: (no net) -> Net-(Q6-Pad3)
- U17 pad 17: (no net) -> Net-(C48-Pad2)
- U17 pad 18: (no net) -> AN0
- U17 pad 19: (no net) -> AN1
- U17 pad 20: (no net) -> AN2
- U17 pad 21: (no net) -> Net-(L6-Pad2)
- U17 pad 22: (no net) -> Net-(R42-Pad2)
- U17 pad 23: (no net) -> Net-(R43-Pad2)
- U17 pad 24: (no net) -> Net-(R44-Pad2)
- U17 pad 25: (no net) -> Net-(U17-Pad25)
- U17 pad 28: (no net) -> Net-(C206-Pad2)
- U17 pad 31: (no net) -> Net-(R41-Pad2)
- U17 pad 33: (no net) -> RW
- U17 pad 8: (no net) -> Net-(R132-Pad2)
- U17 pad 9: (no net) -> Net-(R133-Pad2)
- U18 pad 11: (no net) -> LP
- U18 pad 12: (no net) -> Net-(R132-Pad2)
- U18 pad 13: (no net) -> Net-(R133-Pad2)
- U18 pad 3: (no net) -> BO2
- U18 pad 4: (no net) -> Net-(U18-Pad4)
- U18 pad 5: (no net) -> Net-(U18-Pad4)
- U18 pad 6: (no net) -> O0
- U6 pad 37: (no net) -> OSC
- U6 pad 38: (no net) -> RW
Routing:
- net Net-(R111-Pad2): track 10.2 -> 8.26 mm
- net Net-(R110-Pad2): track 12.9 -> 11.4 mm
- net +5VA: track 660.3 -> 659.0 mm

Commit message: MMU, Joy, Cart and Video
Parts:
- added C102: 1nF, Atari:C_Axial_L5.1mm_D2.5mm_P12.50mm_Horizontal, F.Cu at (46.7, -48.2)
- added C18: 100nF, Atari:C_Axial_L5.1mm_D2.5mm_P12.50mm_Horizontal, F.Cu at (170.2, 33.5)
- added C200: 100nF, Atari:C_Axial_L5.1mm_D2.5mm_P12.50mm_Horizontal, F.Cu at (251.9, 148.3)
- added C201: 100nF, Atari:C_Axial_L5.1mm_D2.5mm_P12.50mm_Horizontal, F.Cu at (251.9, 151.9)
- added C25: 100nF, Atari:C_Axial_L5.1mm_D2.5mm_P12.50mm_Horizontal, F.Cu at (206.5, 74.3)
- added C26: 100nF, Atari:C_Axial_L5.1mm_D2.5mm_P12.50mm_Horizontal, F.Cu at (96.8, 125.8)
- added FB102: Ferrite_Bead, Atari:L_Axial_L7.0mm_D3.3mm_P12.50mm_Horizontal_Fastron_MICC, F.Cu at (304.3, 34.6)
- added FB12: Ferrite_Bead, Atari:L_Axial_L7.0mm_D3.3mm_P12.50mm_Horizontal_Fastron_MICC, F.Cu at (306.9, 26.0)
- added J24: Cartridge, Atari:Cartridge_Slot, F.Cu at (192.1, 29.1)
- added J5: Joystick_Port, Atari:Joystick_Pport, F.Cu at (338.5, 51.3)
- added J6: Joystick_Port, Atari:Joystick_Pport, F.Cu at (338.5, 17.8)
- added L14: 22uH, Atari:L_Axial_L7.0mm_D3.3mm_P12.50mm_Horizontal_Fastron_MICC, F.Cu at (267.5, 149.0)
- added R12: 3k, Atari:R_Axial_DIN0207_L3.6mm_D2.2mm_P10.16mm_Horizontal, F.Cu at (58.4, -13.9)
- added R13: 1k, Atari:R_Axial_DIN0207_L3.6mm_D2.2mm_P10.16mm_Horizontal, F.Cu at (70.2, -28.9)
- added R14: 1k, Atari:R_Axial_DIN0207_L3.6mm_D2.2mm_P10.16mm_Horizontal, F.Cu at (70.2, -25.3)
- added R15: 3k, Atari:R_Axial_DIN0207_L3.6mm_D2.2mm_P10.16mm_Horizontal, F.Cu at (70.2, -21.7)
- added R200: 470k, Atari:R_Axial_DIN0207_L3.6mm_D2.2mm_P10.16mm_Horizontal, F.Cu at (251.9, 162.6)
- added R21: 3k, Atari:R_Axial_DIN0207_L3.6mm_D2.2mm_P10.16mm_Horizontal, F.Cu at (108.6, -15.7)
- added R22: 3k, Atari:R_Axial_DIN0207_L3.6mm_D2.2mm_P10.16mm_Horizontal, F.Cu at (108.6, -12.1)
- added R34: 3k, Atari:R_Axial_DIN0207_L3.6mm_D2.2mm_P10.16mm_Horizontal, F.Cu at (108.6, -8.51)
- added R39: 56k, Atari:R_Axial_DIN0207_L3.6mm_D2.2mm_P10.16mm_Horizontal, F.Cu at (251.9, 155.4)
- added R40: 100, Atari:R_Axial_DIN0207_L3.6mm_D2.2mm_P10.16mm_Horizontal, F.Cu at (251.9, 159.0)
- added U170: LM555, Package_DIP:DIP-8_W7.62mm_Socket, F.Cu at (268.0, 153.5)
- added U2: 74LS138, Package_DIP:DIP-16_W7.62mm_Socket, F.Cu at (206.9, 87.4)
- added U3: MMU, Package_DIP:DIP-20_W7.62mm_Socket, F.Cu at (103.9, 129.4)
- J2: value DIN-5_180degree -> Video
Connections:
- net Net-(R31-Pad2) renamed RNMI
- C205 pad 1: Net-(C205-Pad1) -> RF_VCC
- FB31 pad 1: (no net) -> CHROMA
- FB9 pad 1: (no net) -> MONO
- J2 pad 1: (no net) -> MONO
- J2 pad 2: (no net) -> GND
- J2 pad 4: (no net) -> COMPOSITE
- J2 pad 5: (no net) -> CHROMA
- J4 pad 3: (no net) -> D1XX
- J4 pad 4: (no net) -> MPD
- L13 pad 1: Net-(C205-Pad1) -> RF_VCC
- L23 pad 1: (no net) -> TRIG1
- L30 pad 1: (no net) -> TRIG0
- L32 pad 1: (no net) -> COLOR
- M1 pad 1: (no net) -> COMPOSITE
- M1 pad 2: (no net) -> RF_VCC
- M1 pad 3: (no net) -> COLOR
- M1 pad 4: (no net) -> MONO
- M1 pad 6: (no net) -> GND
- M1 pad 7: (no net) -> GND
- M1 pad 8: (no net) -> GND
- M1 pad 9: (no net) -> GND
- R72 pad 1: +5VA -> +5V
- R73 pad 1: +5VA -> +5V
- U17 pad 11: (no net) -> RD5
- U17 pad 32: (no net) -> GTIA
- U18 pad 10: (no net) -> Net-(U18-Pad10)
- U18 pad 8: (no net) -> GTIA
- U18 pad 9: (no net) -> Net-(U18-Pad10)
- U4 pad 20: (no net) -> BASIC
- U6 pad 4: (no net) -> CASINH

Commit message: Put elements on board
Parts:
- D2, D3: footprint Diode_THT:D_DO-35_SOD27_P7.62mm_Horizontal -> Diode_THT:D_DO-35_SOD27_P12.70mm_Horizontal
- Q1, Q2, Q3: footprint Package_TO_SOT_THT:TO-92 -> Package_TO_SOT_THT:TO-92L_Wide
- moved C102 311.3 mm to (304.0, 127.0), turned to 180 degrees
- moved R12 209.2 mm to (237.0, 95.0), turned to 180 degrees
- moved Q1 186.7 mm to (104.9, 69.4)
- moved C97 182.8 mm to (304.0, 86.0), turned to 180 degrees
- moved R136 176.6 mm to (284.0, 134.0), turned to 180 degrees
- moved C96 171.7 mm to (304.0, 70.0), turned to 180 degrees
- moved R52 170.1 mm to (94.0, 45.5), turned to 90 degrees
- moved D3 167.2 mm to (116.2, 61.7), turned to 90 degrees
- moved L30 165.9 mm to (304.0, 82.0), turned to 180 degrees
- moved R13 165.2 mm to (102.9, 133.0), turned to 180 degrees
- moved R134 164.1 mm to (284.0, 128.0), turned to 180 degrees
- moved D2 162.8 mm to (118.9, 61.7), turned to 90 degrees
- moved R135 162.8 mm to (284.0, 131.0), turned to 180 degrees
- moved L23 160.1 mm to (304.0, 66.0), turned to 180 degrees
- moved R15 158.8 mm to (112.0, 131.5)
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- renumbered U170 to U19
Routing:
- net +5VA: track 659.0 -> 802.1 mm
- net GND: track 261.0 -> 276.7 mm
- net Net-(C111-Pad1): track 0.00 -> 8.00 mm
- net Net-(C111-Pad2): track 0.00 -> 8.00 mm
- net O2: track 73.7 -> 74.7 mm
- net CASMAN: track 92.9 -> 93.8 mm
- net CASBNK: track 70.5 -> 71.5 mm
- net Net-(R110-Pad2): track 11.4 -> 10.6 mm
- net FA14: track 32.6 -> 33.2 mm
- net CAS: track 61.7 -> 62.2 mm
- net FA15: track 32.7 -> 33.2 mm
