File: Atari 130XE.kicad_pcb (KiCad board)
At the start: 2 copper layers, 324 x 204 mm, 184 parts, among them J100 cond, J101 cond, J2 Video, J24 Cartridge, J4 Expansion, J5 Joystick_Port, J6 Joystick_Port, J7 Power, M1 Modulator, Q1 2N3904, Q2 2N3904, Q3 2N3904, Q6 2N3904, SW1 Switch_power_on, U10 DRAM_4464, U11 DRAM_4464, U12 DRAM_4464, U17 GTIA, U18 74LS08, U19 LM555, U2 74LS138, U20 4050, U21 74LS74, U3 MMU, U34 MMMU, U4 BASIC_ROM, U5 27C128, U6 Freddie, U7 Antic, U8 Sally, U9 DRAM_4464, Y1 Crystal, Y2 4,43 MHz

Commit message: PIA and POKEY
Parts:
- added C68: 100nF, Atari:C_Axial_L5.1mm_D2.5mm_P12.50mm_Horizontal, F.Cu at (242.0, 87.0)
- added C69: 100nF, Atari:C_Axial_L5.1mm_D2.5mm_P12.50mm_Horizontal, F.Cu at (234.1, 133.0)
- added C70: 100nF, Atari:C_Axial_L5.1mm_D2.5mm_P12.50mm_Horizontal, F.Cu at (229.0, 148.0)
- added C75: 1nF, Atari:C_Axial_L5.1mm_D2.5mm_P12.50mm_Horizontal, F.Cu at (287.5, 96.0)
- added C76: 1nF, Atari:C_Axial_L5.1mm_D2.5mm_P12.50mm_Horizontal, F.Cu at (287.5, 90.0)
- added C77: 1nF, Atari:C_Axial_L5.1mm_D2.5mm_P12.50mm_Horizontal, F.Cu at (287.5, 102.0)
- added C78: 1nF, Atari:C_Axial_L5.1mm_D2.5mm_P12.50mm_Horizontal, F.Cu at (287.5, 108.0)
- added C79: 22uF, Capacitor_THT:CP_Radial_D5.0mm_P2.50mm, F.Cu at (226.9, 33.4)
- added C80: 1nF, Atari:C_Axial_L5.1mm_D2.5mm_P12.50mm_Horizontal, F.Cu at (217.0, 37.6)
- added C81: 1nF, Atari:C_Axial_L5.1mm_D2.5mm_P12.50mm_Horizontal, F.Cu at (236.0, 45.0)
- added C82: 1nF, Atari:C_Axial_L5.1mm_D2.5mm_P12.50mm_Horizontal, F.Cu at (224.0, 55.7)
- added C83: 1nF, Atari:C_Axial_L5.1mm_D2.5mm_P12.50mm_Horizontal, F.Cu at (228.5, 63.5)
- added C84: 1nF, Atari:C_Axial_L5.1mm_D2.5mm_P12.50mm_Horizontal, F.Cu at (241.0, 50.5)
- added C85: 1nF, Atari:C_Axial_L5.1mm_D2.5mm_P12.50mm_Horizontal, F.Cu at (252.0, 63.0)
- added C86: 1nF, Atari:C_Axial_L5.1mm_D2.5mm_P12.50mm_Horizontal, F.Cu at (249.0, 63.0)
- added C87: 1nF, Atari:C_Axial_L5.1mm_D2.5mm_P12.50mm_Horizontal, F.Cu at (246.0, 63.0)
- added C88: 1nF, Atari:C_Axial_L5.1mm_D2.5mm_P12.50mm_Horizontal, F.Cu at (254.0, 45.0)
- added C89: 1nF, Atari:C_Axial_L5.1mm_D2.5mm_P12.50mm_Horizontal, F.Cu at (252.0, 42.0)
- added C90: 1nF, Atari:C_Axial_L5.1mm_D2.5mm_P12.50mm_Horizontal, F.Cu at (252.0, 39.0)
- added C91: 1nF, Atari:C_Axial_L5.1mm_D2.5mm_P12.50mm_Horizontal, F.Cu at (252.0, 36.0)
- added C92: 1nF, Atari:C_Axial_L5.1mm_D2.5mm_P12.50mm_Horizontal, F.Cu at (252.0, 33.0)
- added C93: 100nF, Atari:C_Axial_L5.1mm_D2.5mm_P12.50mm_Horizontal, F.Cu at (255.1, 174.0)
- added C95: 10nF, Atari:C_Axial_L5.1mm_D2.5mm_P12.50mm_Horizontal, F.Cu at (240.0, 180.0)
- added D5: 1N4148, Diode_THT:D_DO-35_SOD27_P12.70mm_Horizontal, F.Cu at (268.7, 127.4)
- added FB10: Ferrite_Bead, Atari:L_Axial_L7.0mm_D3.3mm_P12.50mm_Horizontal_Fastron_MICC, F.Cu at (229.5, 41.0)
- added FB11: Ferrite_Bead, Atari:L_Axial_L7.0mm_D3.3mm_P12.50mm_Horizontal_Fastron_MICC, F.Cu at (229.5, 45.0)
- added J1: SIO, Atari:SIO_Slot, F.Cu at (283.0, 19.0)
- added J8: Keyboard, Connector_PinHeader_2.54mm:PinHeader_1x24_P2.54mm_Vertical, F.Cu at (237.5, 166.0)
- added L19: 10uH, Atari:L_Axial_L7.0mm_D3.3mm_P12.50mm_Horizontal_Fastron_MICC, F.Cu at (272.0, 33.0)
- added L20: 10uH, Atari:L_Axial_L7.0mm_D3.3mm_P12.50mm_Horizontal_Fastron_MICC, F.Cu at (272.0, 36.8)
- added L21: 10uH, Atari:L_Axial_L7.0mm_D3.3mm_P12.50mm_Horizontal_Fastron_MICC, F.Cu at (272.0, 40.6)
- added L22: 10uH, Atari:L_Axial_L7.0mm_D3.3mm_P12.50mm_Horizontal_Fastron_MICC, F.Cu at (272.0, 44.4)
- added L26: 10uH, Atari:L_Axial_L7.0mm_D3.3mm_P12.50mm_Horizontal_Fastron_MICC, F.Cu at (272.0, 48.2)
- added L27: 10uH, Atari:L_Axial_L7.0mm_D3.3mm_P12.50mm_Horizontal_Fastron_MICC, F.Cu at (272.0, 52.0)
- added L28: 10uH, Atari:L_Axial_L7.0mm_D3.3mm_P12.50mm_Horizontal_Fastron_MICC, F.Cu at (272.0, 55.8)
- added L29: 10uH, Atari:L_Axial_L7.0mm_D3.3mm_P12.50mm_Horizontal_Fastron_MICC, F.Cu at (272.0, 59.6)
- added Q4: 2N3906, Package_TO_SOT_THT:TO-92_Wide, F.Cu at (211.7, 40.8)
- added R117: 100, Atari:R_Axial_DIN0207_L3.6mm_D2.2mm_P10.16mm_Horizontal, F.Cu at (224.0, 60.9)
- added R118: 220, Atari:R_Axial_DIN0207_L3.6mm_D2.2mm_P10.16mm_Horizontal, F.Cu at (228.5, 60.9)
- added R119: 100, Atari:R_Axial_DIN0207_L3.6mm_D2.2mm_P10.16mm_Horizontal, F.Cu at (228.5, 55.7)
- added R120: 220, Atari:R_Axial_DIN0207_L3.6mm_D2.2mm_P10.16mm_Horizontal, F.Cu at (272.8, 67.8)
- added R121: 220, Atari:R_Axial_DIN0207_L3.6mm_D2.2mm_P10.16mm_Horizontal, F.Cu at (270.3, 67.8)
- added R122: 220, Atari:R_Axial_DIN0207_L3.6mm_D2.2mm_P10.16mm_Horizontal, F.Cu at (267.7, 67.8)
- added R123: 220, Atari:R_Axial_DIN0207_L3.6mm_D2.2mm_P10.16mm_Horizontal, F.Cu at (265.2, 67.8)
- added R124: 220, Atari:R_Axial_DIN0207_L3.6mm_D2.2mm_P10.16mm_Horizontal, F.Cu at (262.6, 67.8)
- added R125: 220, Atari:R_Axial_DIN0207_L3.6mm_D2.2mm_P10.16mm_Horizontal, F.Cu at (260.1, 67.8)
- added R126: 220, Atari:R_Axial_DIN0207_L3.6mm_D2.2mm_P10.16mm_Horizontal, F.Cu at (257.6, 67.8)
- added R127: 220, Atari:R_Axial_DIN0207_L3.6mm_D2.2mm_P10.16mm_Horizontal, F.Cu at (255.0, 67.8)
- added R128: 100, Atari:R_Axial_DIN0207_L3.6mm_D2.2mm_P10.16mm_Horizontal, F.Cu at (287.5, 99.0)
- added R129: 100, Atari:R_Axial_DIN0207_L3.6mm_D2.2mm_P10.16mm_Horizontal, F.Cu at (287.5, 93.0)
- added R130: 100, Atari:R_Axial_DIN0207_L3.6mm_D2.2mm_P10.16mm_Horizontal, F.Cu at (287.5, 105.0)
- added R131: 100, Atari:R_Axial_DIN0207_L3.6mm_D2.2mm_P10.16mm_Horizontal, F.Cu at (287.5, 111.0)
- added R137: 270, Atari:R_Axial_DIN0207_L3.6mm_D2.2mm_P10.16mm_Horizontal, F.Cu at (268.5, 132.5)
- added R138: 220, Atari:R_Axial_DIN0207_L3.6mm_D2.2mm_P10.16mm_Horizontal, F.Cu at (284.0, 140.1)
- added R139: 220, Atari:R_Axial_DIN0207_L3.6mm_D2.2mm_P10.16mm_Horizontal, F.Cu at (284.0, 142.6)
- added R140: 220, Atari:R_Axial_DIN0207_L3.6mm_D2.2mm_P10.16mm_Horizontal, F.Cu at (284.0, 137.5)
- added R141: 220, Atari:R_Axial_DIN0207_L3.6mm_D2.2mm_P10.16mm_Horizontal, F.Cu at (284.0, 147.7)
- added R142: 220, Atari:R_Axial_DIN0207_L3.6mm_D2.2mm_P10.16mm_Horizontal, F.Cu at (284.0, 135.0)
- added R143: 220, Atari:R_Axial_DIN0207_L3.6mm_D2.2mm_P10.16mm_Horizontal, F.Cu at (284.0, 150.2)
- added R144: 220, Atari:R_Axial_DIN0207_L3.6mm_D2.2mm_P10.16mm_Horizontal, F.Cu at (284.0, 145.2)
- added R145: 220, Atari:R_Axial_DIN0207_L3.6mm_D2.2mm_P10.16mm_Horizontal, F.Cu at (284.0, 152.8)
- added R146: 220, Atari:R_Axial_DIN0207_L3.6mm_D2.2mm_P10.16mm_Horizontal, F.Cu at (268.5, 137.5)
- added R147: 220, Atari:R_Axial_DIN0207_L3.6mm_D2.2mm_P10.16mm_Horizontal, F.Cu at (268.5, 142.6)
- added R148: 220, Atari:R_Axial_DIN0207_L3.6mm_D2.2mm_P10.16mm_Horizontal, F.Cu at (268.5, 145.2)
- added R149: 220, Atari:R_Axial_DIN0207_L3.6mm_D2.2mm_P10.16mm_Horizontal, F.Cu at (268.5, 140.1)
- added R150: 220, Atari:R_Axial_DIN0207_L3.6mm_D2.2mm_P10.16mm_Horizontal, F.Cu at (268.5, 135.0)
- added R151: 220, Atari:R_Axial_DIN0207_L3.6mm_D2.2mm_P10.16mm_Horizontal, F.Cu at (268.5, 147.7)
- added R152: 220, Atari:R_Axial_DIN0207_L3.6mm_D2.2mm_P10.16mm_Horizontal, F.Cu at (268.5, 152.8)
- added R153: 220, Atari:R_Axial_DIN0207_L3.6mm_D2.2mm_P10.16mm_Horizontal, F.Cu at (268.5, 150.2)
- added R206: 3k3, Atari:R_Axial_DIN0207_L3.6mm_D2.2mm_P10.16mm_Horizontal, F.Cu at (255.0, 84.0)
- added R23: 3k, Atari:R_Axial_DIN0207_L3.6mm_D2.2mm_P10.16mm_Horizontal, F.Cu at (66.0, 149.0)
- added R24: 3k, Atari:R_Axial_DIN0207_L3.6mm_D2.2mm_P10.16mm_Horizontal, F.Cu at (66.0, 143.0)
- added R25: 3k, Atari:R_Axial_DIN0207_L3.6mm_D2.2mm_P10.16mm_Horizontal, F.Cu at (66.0, 146.0)
- added R33: 3k, Atari:R_Axial_DIN0207_L3.6mm_D2.2mm_P10.16mm_Horizontal, F.Cu at (259.0, 109.0)
- added R74: 3k, Atari:R_Axial_DIN0207_L3.6mm_D2.2mm_P10.16mm_Horizontal, F.Cu at (238.4, 107.0)
- added R75: 3k, Atari:R_Axial_DIN0207_L3.6mm_D2.2mm_P10.16mm_Horizontal, F.Cu at (222.0, 131.0)
- added R80: 1k, Atari:R_Axial_DIN0207_L3.6mm_D2.2mm_P10.16mm_Horizontal, F.Cu at (210.6, 107.0)
- added R81: 4k7, Atari:R_Axial_DIN0207_L3.6mm_D2.2mm_P10.16mm_Horizontal, F.Cu at (259.0, 100.0)
- added R82: 4k7, Atari:R_Axial_DIN0207_L3.6mm_D2.2mm_P10.16mm_Horizontal, F.Cu at (259.0, 97.0)
- added R83: 4k7, Atari:R_Axial_DIN0207_L3.6mm_D2.2mm_P10.16mm_Horizontal, F.Cu at (259.0, 103.0)
- added R84: 4k7, Atari:R_Axial_DIN0207_L3.6mm_D2.2mm_P10.16mm_Horizontal, F.Cu at (259.0, 106.0)
- added R85: 3k, Atari:R_Axial_DIN0207_L3.6mm_D2.2mm_P10.16mm_Horizontal, F.Cu at (236.5, 91.0)
- added R86: 3k, Atari:R_Axial_DIN0207_L3.6mm_D2.2mm_P10.16mm_Horizontal, F.Cu at (259.0, 93.0)
- added R87: 3k, Atari:R_Axial_DIN0207_L3.6mm_D2.2mm_P10.16mm_Horizontal, F.Cu at (253.5, 91.0)
- added R88: 3k, Atari:R_Axial_DIN0207_L3.6mm_D2.2mm_P10.16mm_Horizontal, F.Cu at (238.4, 87.0)
- added R89: 47k, Atari:R_Axial_DIN0207_L3.6mm_D2.2mm_P10.16mm_Horizontal, F.Cu at (246.6, 130.4)
- added R90: 100, Atari:R_Axial_DIN0207_L3.6mm_D2.2mm_P10.16mm_Horizontal, F.Cu at (224.0, 156.2)
- added R91: 2k7, Atari:R_Axial_DIN0207_L3.6mm_D2.2mm_P10.16mm_Horizontal, F.Cu at (224.0, 53.1)
- added R92: 4k7, Atari:R_Axial_DIN0207_L3.6mm_D2.2mm_P10.16mm_Horizontal, F.Cu at (224.0, 58.3)
- added R93: 4k7, Atari:R_Axial_DIN0207_L3.6mm_D2.2mm_P10.16mm_Horizontal, F.Cu at (241.0, 58.3)
- added R94: 4k7, Atari:R_Axial_DIN0207_L3.6mm_D2.2mm_P10.16mm_Horizontal, F.Cu at (241.0, 53.1)
- added R95: 1k, Atari:R_Axial_DIN0207_L3.6mm_D2.2mm_P10.16mm_Horizontal, F.Cu at (240.0, 177.0)
- added R96: 47k, Atari:R_Axial_DIN0207_L3.6mm_D2.2mm_P10.16mm_Horizontal, F.Cu at (256.0, 129.9)
- added U22: POKEY, Package_DIP:DIP-40_W15.24mm_Socket, F.Cu at (203.0, 127.0)
- added U23: PIA, Package_DIP:DIP-40_W15.24mm_Socket, F.Cu at (203.0, 83.0)
- added U24: CD4051B, Package_DIP:DIP-18_W7.62mm_Socket, F.Cu at (229.0, 145.0)
- added U25: CD4051B, Package_DIP:DIP-18_W7.62mm_Socket, F.Cu at (229.0, 158.6)
- added W1: 0, Atari:R_Axial_DIN0207_L3.6mm_D2.2mm_P10.16mm_Horizontal, F.Cu at (209.5, 134.0)
- moved C18 44.7 mm to (211.5, 50.5)
- moved J5 32.0 mm to (313.0, 3.00)
- moved J6 32.0 mm to (313.0, 35.0)
- moved C25 21.7 mm to (185.2, 78.7)
- moved R136 1.54 mm to (284.0, 132.5)
- moved R12 1.12 mm to (236.5, 94.0)
- moved R19 1.12 mm to (271.5, 112.0)
- moved R135 1.08 mm to (284.0, 129.9)
- moved R134 0.63 mm to (284.0, 127.4)
Connections:
- J2 pad 3: (no net) -> AUDIO
- J5 pad 1: (no net) -> FWD1
- J5 pad 2: (no net) -> BACK1
- J5 pad 3: (no net) -> LEFT1
- J5 pad 4: (no net) -> RIGHT1
- J6 pad 1: (no net) -> FWD0
- J6 pad 2: (no net) -> BACK0
- J6 pad 3: (no net) -> LEFT0
- J6 pad 4: (no net) -> RIGHT0
- L14 pad 2: (no net) -> RESET
- R134 pad 1: (no net) -> START
- R135 pad 1: (no net) -> SELECT
- R136 pad 1: (no net) -> OPTION
- U2 pad 12: (no net) -> PIA
- U2 pad 13: (no net) -> POKEY
- U3 pad 18: (no net) -> PB1
- U3 pad 6: (no net) -> PB7
- U3 pad 9: (no net) -> PB0
- U34 pad 14: (no net) -> PB5
- U34 pad 3: (no net) -> PB2
- U34 pad 4: (no net) -> PB3
- U34 pad 5: (no net) -> PB4
Routing:
- net PB2: track 0.00 -> 17.0 mm
- net PB3: track 0.00 -> 13.3 mm
- net +5VA: track 802.1 -> 815.0 mm
- net PB4: track 0.00 -> 9.39 mm

Commit message: Pokey finish
Parts:
- added C63: 47nF, Atari:C_Axial_L5.1mm_D2.5mm_P12.50mm_Horizontal, F.Cu at (377.1, 114.1)
- added C64: 47nF, Atari:C_Axial_L5.1mm_D2.5mm_P12.50mm_Horizontal, F.Cu at (345.8, 118.9)
- added C65: 47nF, Atari:C_Axial_L5.1mm_D2.5mm_P12.50mm_Horizontal, F.Cu at (361.4, 114.1)
- added C66: 47nF, Atari:C_Axial_L5.1mm_D2.5mm_P12.50mm_Horizontal, F.Cu at (345.8, 122.5)
- added C71: 1nF, Atari:C_Axial_L5.1mm_D2.5mm_P12.50mm_Horizontal, F.Cu at (361.4, 117.6)
- added C72: 1nF, Atari:C_Axial_L5.1mm_D2.5mm_P12.50mm_Horizontal, F.Cu at (345.8, 126.0)
- added C73: 1nF, Atari:C_Axial_L5.1mm_D2.5mm_P12.50mm_Horizontal, F.Cu at (345.8, 129.6)
- added C74: 1nF, Atari:C_Axial_L5.1mm_D2.5mm_P12.50mm_Horizontal, F.Cu at (345.8, 133.1)
- added C98: 10uF, Capacitor_THT:CP_Radial_Tantal_D5.0mm_P2.50mm, F.Cu at (377.6, 134.7)
- added C99: 1nF, Atari:C_Axial_L5.1mm_D2.5mm_P12.50mm_Horizontal, F.Cu at (345.8, 136.7)
- added L15: 10uH, Atari:L_Axial_L7.0mm_D3.3mm_P12.50mm_Horizontal_Fastron_MICC, F.Cu at (345.8, 114.7)
- added L16: 10uH, Atari:L_Axial_L7.0mm_D3.3mm_P12.50mm_Horizontal_Fastron_MICC, F.Cu at (361.4, 121.8)
- added L17: 10uH, Atari:L_Axial_L7.0mm_D3.3mm_P12.50mm_Horizontal_Fastron_MICC, F.Cu at (361.4, 126.7)
- added L18: 10uH, Atari:L_Axial_L7.0mm_D3.3mm_P12.50mm_Horizontal_Fastron_MICC, F.Cu at (377.1, 118.3)
- added L24: 10uH, Atari:L_Axial_L7.0mm_D3.3mm_P12.50mm_Horizontal_Fastron_MICC, F.Cu at (361.4, 131.5)
- added R76: 1k8, Atari:R_Axial_DIN0207_L3.6mm_D2.2mm_P10.16mm_Horizontal, F.Cu at (361.4, 135.7)
- added R77: 1k8, Atari:R_Axial_DIN0207_L3.6mm_D2.2mm_P10.16mm_Horizontal, F.Cu at (377.1, 122.5)
- added R78: 1k8, Atari:R_Axial_DIN0207_L3.6mm_D2.2mm_P10.16mm_Horizontal, F.Cu at (377.1, 126.1)
- added R79: 1k8, Atari:R_Axial_DIN0207_L3.6mm_D2.2mm_P10.16mm_Horizontal, F.Cu at (377.1, 129.7)
Connections:
- C1 pad 2: GND -> JOY_GND
- C10 pad 2: GND -> JOY_GND
- C102 pad 2: GND -> JOY_GND
- C103 pad 2: GND -> JOY_GND
- C11 pad 2: GND -> JOY_GND
- C12 pad 2: GND -> JOY_GND
- C13 pad 2: GND -> JOY_GND
- C14 pad 2: GND -> JOY_GND
- C15 pad 2: GND -> JOY_GND
- C18 pad 2: GND -> JOY_GND
- C2 pad 2: GND -> JOY_GND
- C201 pad 2: GND -> JOY_GND
- C205 pad 2: GND -> JOY_GND
- C206 pad 1: GND -> JOY_GND
- C25 pad 2: GND -> JOY_GND
- C26 pad 2: GND -> JOY_GND
- C27 pad 2: GND -> JOY_GND
- C28 pad 2: GND -> JOY_GND
- C29 pad 2: GND -> JOY_GND
- C3 pad 2: GND -> JOY_GND
- C30 pad 2: GND -> JOY_GND
- C31 pad 2: GND -> JOY_GND
- C32 pad 2: GND -> JOY_GND
- C33 pad 2: GND -> JOY_GND
- C34 pad 2: GND -> JOY_GND
- C35 pad 2: GND -> JOY_GND
- C36 pad 2: GND -> JOY_GND
- C37 pad 2: GND -> JOY_GND
- C4 pad 2: GND -> JOY_GND
- C42 pad 2: GND -> JOY_GND
- C46 pad 1: GND -> JOY_GND
- C47 pad 1: GND -> JOY_GND
- C48 pad 1: GND -> JOY_GND
- C5 pad 2: GND -> JOY_GND
- C50 pad 2: GND -> JOY_GND
- C51 pad 2: GND -> JOY_GND
- C6 pad 2: GND -> JOY_GND
- C60 pad 1: GND -> JOY_GND
- C61 pad 1: GND -> JOY_GND
- C68 pad 2: GND -> JOY_GND
- C69 pad 2: GND -> JOY_GND
- C7 pad 2: GND -> JOY_GND
- C70 pad 2: GND -> JOY_GND
- C75 pad 2: GND -> JOY_GND
- C76 pad 2: GND -> JOY_GND
- C77 pad 2: GND -> JOY_GND
- C78 pad 2: GND -> JOY_GND
- C79 pad 2: GND -> JOY_GND
- C8 pad 2: GND -> JOY_GND
- C80 pad 2: GND -> JOY_GND
- C81 pad 2: GND -> JOY_GND
- C82 pad 2: GND -> JOY_GND
- C83 pad 2: GND -> JOY_GND
- C84 pad 2: GND -> JOY_GND
- C85 pad 2: GND -> JOY_GND
- C86 pad 2: GND -> JOY_GND
- C87 pad 2: GND -> JOY_GND
- C88 pad 2: GND -> JOY_GND
- C89 pad 2: GND -> JOY_GND
- C9 pad 2: GND -> JOY_GND
- C90 pad 2: GND -> JOY_GND
- C91 pad 2: GND -> JOY_GND
- C92 pad 2: GND -> JOY_GND
- C93 pad 2: GND -> JOY_GND
- C95 pad 2: GND -> JOY_GND
- C96 pad 1: GND -> JOY_GND
- C97 pad 1: GND -> JOY_GND
- Ek1 pad 1: GND -> JOY_GND
- Ek2 pad 1: GND -> JOY_GND
- Ek3 pad 1: GND -> JOY_GND
- Ek4 pad 1: GND -> JOY_GND
- Ek5 pad 1: GND -> JOY_GND
- Ek6 pad 1: GND -> JOY_GND
- Ek7 pad 1: GND -> JOY_GND
- J1 pad 12: (no net) -> Net-(J1-Pad12)
- J1 pad 4: GND -> JOY_GND
- J1 pad 6: GND -> JOY_GND
- J100 pad 1: GND -> JOY_GND
- J101 pad 1: GND -> JOY_GND
- J2 pad 2: GND -> JOY_GND
- J24 pad B: GND -> JOY_GND
- J4 pad H: GND -> JOY_GND
- J5 pad 5: (no net) -> POT_B1
- J5 pad 8: GND -> JOY_GND
- J5 pad 9: (no net) -> POT_A1
- J6 pad 5: (no net) -> POT_B0
- J6 pad 8: GND -> JOY_GND
- J6 pad 9: (no net) -> POT_A0
- J7 pad 2: GND -> JOY_GND
- J7 pad 3: GND -> JOY_GND
- J7 pad 5: GND -> JOY_GND
- J7 pad 7: GND -> JOY_GND
- J8 pad 3: GND -> JOY_GND
- M1 pad 6: GND -> JOY_GND
- M1 pad 7: GND -> JOY_GND
- M1 pad 8: GND -> JOY_GND
- M1 pad 9: GND -> JOY_GND
- Q1 pad 1: GND -> JOY_GND
- Q6 pad 1: GND -> JOY_GND
- R13 pad 2: GND -> JOY_GND
- R14 pad 2: GND -> JOY_GND
- R200 pad 2: GND -> JOY_GND
- R202 pad 1: GND -> JOY_GND
- R52 pad 2: GND -> JOY_GND
- R53 pad 2: GND -> JOY_GND
- R69 pad 2: GND -> JOY_GND
- R90 pad 2: GND -> JOY_GND
- RV38 pad 3: GND -> JOY_GND
- U10 pad 1: GND -> JOY_GND
- U10 pad 18: GND -> JOY_GND
- U11 pad 1: GND -> JOY_GND
- U11 pad 18: GND -> JOY_GND
- U12 pad 1: GND -> JOY_GND
- U12 pad 18: GND -> JOY_GND
- U17 pad 3: GND -> JOY_GND
- U19 pad 1: GND -> JOY_GND
- U2 pad 5: GND -> JOY_GND
- U2 pad 8: GND -> JOY_GND
- U20 pad 8: GND -> JOY_GND
- U20 pad 9: GND -> JOY_GND
- U22 pad 1: (no net) -> JOY_GND
- U22 pad 11: GND -> JOY_GND
- U22 pad 12: (no net) -> Net-(C66-Pad1)
- U22 pad 13: (no net) -> Net-(C63-Pad1)
- U22 pad 14: (no net) -> Net-(C65-Pad1)
- U22 pad 15: (no net) -> Net-(C64-Pad1)
- U22 pad 17: (no net) -> +5P
- U22 pad 8: GND -> JOY_GND
- U22 pad 9: GND -> JOY_GND
- U23 pad 1: GND -> JOY_GND
- U24 pad 6: GND -> JOY_GND
- U24 pad 7: GND -> JOY_GND
- U24 pad 8: GND -> JOY_GND
- U25 pad 6: GND -> JOY_GND
- U25 pad 7: GND -> JOY_GND
- U25 pad 8: GND -> JOY_GND
- U3 pad 10: GND -> JOY_GND
- U34 pad 7: GND -> JOY_GND
- U34 pad 8: GND -> JOY_GND
- U4 pad 12: GND -> JOY_GND
- U5 pad 14: GND -> JOY_GND
- U6 pad 20: GND -> JOY_GND
- U7 pad 1: GND -> JOY_GND
- U8 pad 1: GND -> JOY_GND
- U8 pad 21: GND -> JOY_GND
- U8 pad 38: GND -> JOY_GND
- U8 pad 5: GND -> JOY_GND
- U9 pad 1: GND -> JOY_GND
- U9 pad 18: GND -> JOY_GND
- W1 pad 2: GND -> JOY_GND
Routing:
- net JOY_GND: track 0.00 -> 276.7 mm, vias 0 -> 2
- net GND: track 276.7 -> 0.00 mm, vias 2 -> 0
- added copper zone on F.Cu, net (none)
- added copper zone on F.Cu, net Net-(J1-Pad12)
- added copper zone on B.Cu, net POT_A0
- removed copper zone on B.Cu, net GND

Commit message: Schema finished
Parts:
- removed C99: 1nF, Atari:C_Axial_L5.1mm_D2.5mm_P12.50mm_Horizontal
- removed L24: 10uH, Atari:L_Axial_L7.0mm_D3.3mm_P12.50mm_Horizontal_Fastron_MICC
- added C43: 100nF, Atari:C_Axial_L5.1mm_D2.5mm_P12.50mm_Horizontal, F.Cu at (242.7, 106.5)
- added C62: 1nF, Atari:C_Axial_L5.1mm_D2.5mm_P12.50mm_Horizontal, F.Cu at (304.0, 121.0)
- added C94: 10nF, Atari:C_Axial_L5.1mm_D2.5mm_P12.50mm_Horizontal, F.Cu at (227.5, 174.0)
- added L25: 10uH, Atari:L_Axial_L7.0mm_D3.3mm_P12.50mm_Horizontal_Fastron_MICC, F.Cu at (304.0, 134.0)
- C98: footprint Capacitor_THT:CP_Radial_Tantal_D5.0mm_P2.50mm -> Capacitor_THT:C_Axial_L12.0mm_D6.5mm_P15.00mm_Horizontal
- U24, U25: footprint Package_DIP:DIP-18_W7.62mm_Socket -> Package_DIP:DIP-16_W7.62mm_Socket
- moved C74 113.9 mm to (288.0, 35.0), turned to 180 degrees
- moved C73 113.4 mm to (288.0, 32.0), turned to 180 degrees
- moved L16 105.7 mm to (291.0, 43.0), turned to 180 degrees
- moved L15 93.4 mm to (291.0, 39.0), turned to 180 degrees
- moved C98 89.3 mm to (289.0, 146.3)
- moved C63 86.4 mm to (291.5, 102.0)
- moved L18 85.7 mm to (304.0, 73.5), turned to 180 degrees
- moved C71 83.1 mm to (288.5, 77.7), turned to 180 degrees
- moved R79 81.7 mm to (304.0, 93.0), turned to 180 degrees
- moved R78 81.5 mm to (304.0, 90.0), turned to 180 degrees
- moved R77 77.7 mm to (304.0, 96.0), turned to 180 degrees
- moved C72 77.7 mm to (288.5, 73.5), turned to 180 degrees
- moved L17 75.5 mm to (304.0, 77.7), turned to 180 degrees
- moved C65 70.2 mm to (291.5, 108.0)
- moved R76 68.2 mm to (304.0, 99.0), turned to 180 degrees
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Connections:
- C1 pad 2: JOY_GND -> GND
- C10 pad 2: JOY_GND -> GND
- C102 pad 1: +5P -> Net-(C102-Pad1)
- C102 pad 2: JOY_GND -> GND
- C103 pad 2: JOY_GND -> GND
- C11 pad 2: JOY_GND -> GND
- C12 pad 2: JOY_GND -> GND
- C13 pad 2: JOY_GND -> GND
- C14 pad 2: JOY_GND -> GND
- C15 pad 2: JOY_GND -> GND
- C18 pad 2: JOY_GND -> GND
- C2 pad 2: JOY_GND -> GND
- C201 pad 1: +5V -> +5VA
- C201 pad 2: JOY_GND -> GND
- C205 pad 2: JOY_GND -> GND
- C206 pad 1: JOY_GND -> GND
- C25 pad 1: +5P -> +5VA
- C25 pad 2: JOY_GND -> GND
- C26 pad 2: JOY_GND -> GND
- C27 pad 2: JOY_GND -> GND
- C28 pad 2: JOY_GND -> GND
- C29 pad 2: JOY_GND -> GND
- C3 pad 2: JOY_GND -> GND
- C30 pad 2: JOY_GND -> GND
- C31 pad 2: JOY_GND -> GND
- C32 pad 2: JOY_GND -> GND
- C33 pad 2: JOY_GND -> GND
- C34 pad 2: JOY_GND -> GND
- C35 pad 2: JOY_GND -> GND
- C36 pad 2: JOY_GND -> GND
- C37 pad 2: JOY_GND -> GND
- C4 pad 2: JOY_GND -> GND
- C42 pad 2: JOY_GND -> GND
- C46 pad 1: JOY_GND -> GND
- C47 pad 1: JOY_GND -> GND
- C48 pad 1: JOY_GND -> GND
- C5 pad 2: JOY_GND -> GND
- C50 pad 2: JOY_GND -> GND
- C51 pad 2: JOY_GND -> GND
- C6 pad 2: JOY_GND -> GND
- C60 pad 1: JOY_GND -> GND
- C61 pad 1: JOY_GND -> GND
- C63 pad 2: JOY_GND -> GND
- C64 pad 2: JOY_GND -> GND
- C65 pad 2: JOY_GND -> GND
- C66 pad 2: JOY_GND -> GND
- C68 pad 2: JOY_GND -> GND
- C69 pad 2: JOY_GND -> GND
- C7 pad 2: JOY_GND -> GND
- C70 pad 1: Net-(C70-Pad1) -> +5VA
- C70 pad 2: JOY_GND -> GND
- C71 pad 2: JOY_GND -> GND
- C72 pad 2: JOY_GND -> GND
- C73 pad 2: JOY_GND -> GND
- C74 pad 2: JOY_GND -> GND
- C75 pad 2: JOY_GND -> GND
- C76 pad 2: JOY_GND -> GND
- C77 pad 2: JOY_GND -> GND
- C78 pad 2: JOY_GND -> GND
- C79 pad 2: JOY_GND -> GND
- C8 pad 2: JOY_GND -> GND
- C80 pad 2: JOY_GND -> GND
- C81 pad 2: JOY_GND -> GND
- C82 pad 2: JOY_GND -> GND
- C83 pad 2: JOY_GND -> GND
- C84 pad 2: JOY_GND -> GND
- C85 pad 2: JOY_GND -> GND
- C86 pad 2: JOY_GND -> GND
- C87 pad 2: JOY_GND -> GND
- C88 pad 2: JOY_GND -> GND
- C89 pad 2: JOY_GND -> GND
- C9 pad 2: JOY_GND -> GND
- C90 pad 2: JOY_GND -> GND
- C91 pad 2: JOY_GND -> GND
- C92 pad 2: JOY_GND -> GND
- C93 pad 2: JOY_GND -> GND
- C95 pad 2: JOY_GND -> GND
- C96 pad 1: JOY_GND -> GND
- C97 pad 1: JOY_GND -> GND
- C98 pad 2: JOY_GND -> GND
- Ek1 pad 1: JOY_GND -> GND
- Ek2 pad 1: JOY_GND -> GND
- Ek3 pad 1: JOY_GND -> GND
- Ek4 pad 1: JOY_GND -> GND
- Ek5 pad 1: JOY_GND -> GND
- Ek6 pad 1: JOY_GND -> GND
- Ek7 pad 1: JOY_GND -> GND
- FB102 pad 1: Net-(FB102-Pad1) -> Net-(C102-Pad1)
- FB102 pad 2: +5P -> Net-(FB102-Pad2)
- J1 pad 12: Net-(J1-Pad12) -> (no net)
- J1 pad 4: JOY_GND -> GND
- J1 pad 6: JOY_GND -> GND
- J100 pad 1: JOY_GND -> GND
- J101 pad 1: JOY_GND -> GND
- J2 pad 2: JOY_GND -> GND
- J24 pad B: JOY_GND -> GND
- J4 pad H: JOY_GND -> GND
- J5 pad 7: Net-(FB102-Pad1) -> Net-(C102-Pad1)
- J5 pad 8: JOY_GND -> GND
- J6 pad 7: Net-(FB102-Pad1) -> Net-(C102-Pad1)
- J6 pad 8: JOY_GND -> GND
- J7 pad 2: JOY_GND -> GND
- J7 pad 3: JOY_GND -> GND
- J7 pad 5: JOY_GND -> GND
- J7 pad 7: JOY_GND -> GND
- J8 pad 3: JOY_GND -> GND
- M1 pad 6: JOY_GND -> GND
- M1 pad 7: JOY_GND -> GND
- M1 pad 8: JOY_GND -> GND
- M1 pad 9: JOY_GND -> GND
- Q1 pad 1: JOY_GND -> GND
- Q6 pad 1: JOY_GND -> GND
- R12 pad 1: +5P -> +5VA
- R13 pad 2: JOY_GND -> GND
- R14 pad 2: JOY_GND -> GND
- R200 pad 2: JOY_GND -> GND
- R202 pad 1: JOY_GND -> GND
- R39 pad 1: +5V -> +5VA
- R52 pad 2: JOY_GND -> GND
- R53 pad 2: JOY_GND -> GND
- R69 pad 2: JOY_GND -> GND
- R80 pad 2: +5P -> +5VA
- R90 pad 2: JOY_GND -> GND
- RV38 pad 3: JOY_GND -> GND
- U10 pad 1: JOY_GND -> GND
- U10 pad 18: JOY_GND -> GND
- U11 pad 1: JOY_GND -> GND
- U11 pad 18: JOY_GND -> GND
- U12 pad 1: JOY_GND -> GND
- U12 pad 18: JOY_GND -> GND
- U17 pad 3: JOY_GND -> GND
- U18 pad 14: (no net) -> +5VA
- U18 pad 7: (no net) -> GND
- U19 pad 1: JOY_GND -> GND
- U19 pad 4: +5V -> +5VA
- U19 pad 8: +5V -> +5VA
- U2 pad 16: +5P -> +5VA
- U2 pad 5: JOY_GND -> GND
- U2 pad 8: JOY_GND -> GND
- U20 pad 8: JOY_GND -> GND
- U20 pad 9: JOY_GND -> GND
- U22 pad 1: JOY_GND -> GND
- U22 pad 11: JOY_GND -> GND
- U22 pad 8: JOY_GND -> GND
- U22 pad 9: JOY_GND -> GND
- U23 pad 1: JOY_GND -> GND
- U24 pad 6: JOY_GND -> GND
- U24 pad 7: JOY_GND -> GND
- U24 pad 8: JOY_GND -> GND
- U25 pad 16: Net-(C70-Pad1) -> +5VA
- U25 pad 6: JOY_GND -> GND
- U25 pad 7: JOY_GND -> GND
- U25 pad 8: JOY_GND -> GND
- U3 pad 10: JOY_GND -> GND
- U34 pad 7: JOY_GND -> GND
- U34 pad 8: JOY_GND -> GND
- U4 pad 12: JOY_GND -> GND
- U5 pad 14: JOY_GND -> GND
- U6 pad 20: JOY_GND -> GND
- U7 pad 1: JOY_GND -> GND
- U8 pad 1: JOY_GND -> GND
- U8 pad 21: JOY_GND -> GND
- U8 pad 38: JOY_GND -> GND
- U8 pad 5: JOY_GND -> GND
- U9 pad 1: JOY_GND -> GND
- U9 pad 18: JOY_GND -> GND
- W1 pad 2: JOY_GND -> GND
Routing:
- net GND: track 0.00 -> 803.3 mm, vias 0 -> 4
- net +5VA: track 815.0 -> 1224.3 mm, vias 6 -> 8
- net JOY_GND: track 276.7 -> 0.00 mm, vias 2 -> 0
- net Net-(C102-Pad1): track 0.00 -> 119.5 mm
- net +5P: track 0.00 -> 107.7 mm
- net Net-(C200-Pad1): track 0.00 -> 25.8 mm
- net Net-(R75-Pad1): track 0.00 -> 19.9 mm
- net Net-(C95-Pad1): track 0.00 -> 15.0 mm
- net Net-(FB102-Pad2): track 0.00 -> 14.1 mm
- net RESET: track 0.00 -> 8.01 mm
- net Net-(C200-Pad2): track 0.00 -> 7.36 mm
- removed copper zone on F.Cu, net Net-(J1-Pad12)
