File: Atari 130XE.kicad_pcb (KiCad board)
At the start: 2 copper layers, 324 x 204 mm, 303 parts, among them J1 SIO, J100 cond, J101 cond, J2 Video, J24 Cartridge, J4 Expansion, J5 Joystick_Port, J6 Joystick_Port, J7 Power, J8 Keyboard, M1 Modulator, Q1 2N3904, Q2 2N3904, Q3 2N3904, Q4 2N3906, Q6 2N3904, SW1 Switch_power_on, U10 DRAM_4464, U11 DRAM_4464, U12 DRAM_4464, U17 GTIA, U18 74LS08, U19 LM555, U2 74LS138, U20 4050, U21 74LS74, U22 POKEY, U23 PIA, U24 CD4051B, U25 CD4051B, U3 MMU, U34 MMMU, U4 BASIC_ROM, U5 27C128, U6 Freddie, U7 Antic, U8 Sally, U9 DRAM_4464, Y1 Crystal, Y2 4,43 MHz

Commit message: Audio
Parts:
- added C112: 1nF, Atari:C_Axial_L5.1mm_D2.5mm_P12.50mm_Horizontal, F.Cu at (333.8, 117.0)
- added C16: 1nF, Atari:C_Axial_L5.1mm_D2.5mm_P12.50mm_Horizontal, F.Cu at (333.8, 120.6)
- added C17: 47nF, Atari:C_Axial_L5.1mm_D2.5mm_P12.50mm_Horizontal, F.Cu at (349.5, 117.0)
- added C19: 4,7uF, Capacitor_THT:CP_Radial_D8.0mm_P3.50mm, F.Cu at (376.5, 139.0)
- added C20: 4,7uF, Capacitor_THT:CP_Radial_D8.0mm_P3.50mm, F.Cu at (366.8, 139.0)
- added C21: 1nF, Atari:C_Axial_L5.1mm_D2.5mm_P12.50mm_Horizontal, F.Cu at (333.8, 124.1)
- added C23: 47nF, Atari:C_Axial_L5.1mm_D2.5mm_P12.50mm_Horizontal, F.Cu at (349.5, 120.6)
- added C24: 10uF, Capacitor_THT:C_Axial_L12.0mm_D6.5mm_P15.00mm_Horizontal, F.Cu at (63.2, 109.4)
- added R1: 2k2, Atari:R_Axial_DIN0207_L3.6mm_D2.2mm_P10.16mm_Horizontal, F.Cu at (349.5, 124.1)
- added R10: 1k, Atari:R_Axial_DIN0207_L3.6mm_D2.2mm_P10.16mm_Horizontal, F.Cu at (365.1, 120.6)
- added R11: 2k2, Atari:R_Axial_DIN0207_L3.6mm_D2.2mm_P10.16mm_Horizontal, F.Cu at (333.8, 142.0)
- added R2: 1k, Atari:R_Axial_DIN0207_L3.6mm_D2.2mm_P10.16mm_Horizontal, F.Cu at (349.5, 127.7)
- added R3: 6k2, Atari:R_Axial_DIN0207_L3.6mm_D2.2mm_P10.16mm_Horizontal, F.Cu at (349.5, 131.3)
- added R4: 56k, Atari:R_Axial_DIN0207_L3.6mm_D2.2mm_P10.16mm_Horizontal, F.Cu at (349.5, 134.9)
- added R5: 470k, Atari:R_Axial_DIN0207_L3.6mm_D2.2mm_P10.16mm_Horizontal, F.Cu at (333.8, 127.7)
- added R6: 68k, Atari:R_Axial_DIN0207_L3.6mm_D2.2mm_P10.16mm_Horizontal, F.Cu at (79.9, 72.2)
- added R7: 2k, Atari:R_Axial_DIN0207_L3.6mm_D2.2mm_P10.16mm_Horizontal, F.Cu at (63.3, 70.9)
- added R8: 5k1, Atari:R_Axial_DIN0207_L3.6mm_D2.2mm_P10.16mm_Horizontal, F.Cu at (365.1, 117.0)
- added R9: 3k3, Atari:R_Axial_DIN0207_L3.6mm_D2.2mm_P10.16mm_Horizontal, F.Cu at (333.8, 138.5)
- added U1: LM358, Package_DIP:DIP-8_W7.62mm_Socket, F.Cu at (66.0, 67.7)
Connections:
- J1 pad 11: (no net) -> SIOAUDIO
- M1 pad 5: (no net) -> Net-(M1-Pad5)
- U17 pad 15: (no net) -> BELL

Commit message: Audio put on board
Parts:
- added C204: 100nF, Atari:C_Axial_L5.1mm_D2.5mm_P12.50mm_Horizontal, F.Cu at (87.4, 60.4)
- C24, C98: footprint Capacitor_THT:C_Axial_L12.0mm_D6.5mm_P15.00mm_Horizontal -> Capacitor_THT:CP_Axial_L11.0mm_D6.0mm_P18.00mm_Horizontal
- moved C19 302.6 mm to (76.9, 96.9)
- moved C20 301.5 mm to (68.2, 96.9)
- moved R3 291.2 mm to (63.0, 79.0), turned to 270 degrees
- moved R8 289.5 mm to (81.7, 58.0), turned to 270 degrees
- moved R10 287.6 mm to (84.4, 58.0), turned to 270 degrees
- moved R2 285.3 mm to (66.5, 91.5), turned to 90 degrees
- moved R1 283.1 mm to (70.0, 79.0), turned to 270 degrees
- moved R4 281.0 mm to (70.0, 105.3)
- moved C16 281.0 mm to (60.5, 55.4), turned to 180 degrees
- moved C17 279.6 mm to (70.0, 108.0)
- moved R9 274.0 mm to (67.0, 76.0)
- moved R11 271.4 mm to (64.1, 112.0), turned to 90 degrees
- moved C21 264.2 mm to (73.5, 79.0), turned to 270 degrees
- moved C23 252.9 mm to (100.9, 73.9), turned to 270 degrees
- moved C112 251.7 mm to (82.5, 102.7), turned to 180 degrees
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Connections:
- C16 pad 2: +5VA -> +5C
- C17 pad 2: (no net) -> SOUND
- R80 pad 1: AUDIO -> SOUND
- R9 pad 1: +5VA -> +5C
- RV38 pad 1: Net-(C47-Pad2) -> GND
- RV38 pad 3: GND -> Net-(C47-Pad2)
- U1 pad 8: +5VA -> +5C
- U22 pad 37: AUDIO -> SOUND
- U24 pad 11: K2 -> K0
- U24 pad 9: K0 -> K2
Routing:
- net Net-(L14-Pad1): track 0.00 -> 81.6 mm, vias 0 -> 2
- net Net-(R139-Pad2): track 0.00 -> 74.1 mm, vias 0 -> 1
- net Net-(R141-Pad2): track 0.00 -> 73.0 mm, vias 0 -> 1
- net Net-(R138-Pad2): track 0.00 -> 70.1 mm, vias 0 -> 1
- net Net-(R140-Pad2): track 0.00 -> 68.1 mm, vias 0 -> 1
- net BSC: track 0.00 -> 64.0 mm, vias 0 -> 1
- net Net-(R144-Pad2): track 0.00 -> 60.9 mm, vias 0 -> 1
- net Net-(R142-Pad2): track 0.00 -> 60.5 mm
- net OUT3: track 0.00 -> 60.0 mm
- net IN4: track 0.00 -> 59.3 mm, vias 0 -> 1
- net Net-(R143-Pad2): track 0.00 -> 58.2 mm, vias 0 -> 1
- net OUT5: track 0.00 -> 55.6 mm
- net IN0: track 0.00 -> 52.0 mm, vias 0 -> 1
- net OUT7: track 0.00 -> 51.2 mm
- net IN3: track 0.00 -> 47.2 mm, vias 0 -> 1
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
Commit message: Patching
Parts:
- moved R133 12.5 mm to (288.5, 66.0), turned to 180 degrees
- moved R80 0.26 mm to (210.9, 108.0)
Connections:
- C58 pad 2: Net-(C58-Pad2) -> GND
- R73 pad 1: +5V -> +5VA
- U21 pad 7: Net-(C58-Pad2) -> GND
- U22 pad 7: O2 -> BO2
- U23 pad 25: O2 -> BO2
- Y2 pad 1: Net-(C59-Pad2) -> Net-(C111-Pad1)
- Y2 pad 2: Net-(C111-Pad1) -> Net-(C59-Pad2)
Routing:
- net GND: track 816.9 -> 1090.2 mm
- net OSC: track 0.00 -> 130.4 mm, vias 0 -> 2
- net Net-(R136-Pad2): track 0.00 -> 125.1 mm, vias 0 -> 1
- net Net-(R135-Pad2): track 0.00 -> 123.3 mm, vias 0 -> 1
- net Net-(R134-Pad2): track 0.00 -> 121.3 mm, vias 0 -> 1
- net Net-(C63-Pad1): track 0.00 -> 99.8 mm, vias 0 -> 2
- net Net-(C66-Pad1): track 0.00 -> 97.9 mm, vias 0 -> 2
- net BO2: track 0.00 -> 90.0 mm, vias 0 -> 1
- net Net-(C65-Pad1): track 0.00 -> 87.1 mm, vias 0 -> 1
- net Net-(C64-Pad1): track 0.00 -> 80.2 mm, vias 0 -> 1
- net +5VA: track 1221.8 -> 1299.6 mm
- net Net-(R120-Pad2): track 0.00 -> 72.6 mm
- net D2: track 28.1 -> 100.6 mm
- net D7: track 28.1 -> 98.3 mm
- net D6: track 28.1 -> 97.4 mm
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
Commit message: tracking
Parts:
- moved C30 12.5 mm to (144.2, 89.0), turned to 180 degrees
- moved C31 12.5 mm to (144.2, 63.0), turned to 180 degrees
Routing:
- net D3: track 96.7 -> 234.7 mm, vias 0 -> 4
- net +5VA: track 1299.6 -> 1427.7 mm, vias 8 -> 10
- net D4: track 96.8 -> 202.1 mm, vias 0 -> 2
- net D5: track 96.7 -> 196.1 mm, vias 0 -> 2
- net DATA_OUT: track 3.00 -> 102.1 mm, vias 0 -> 1
- net D6: track 97.4 -> 193.1 mm, vias 0 -> 1
- net DATA_IN: track 3.00 -> 94.2 mm, vias 0 -> 1
- net CLK_OUT: track 3.00 -> 90.1 mm, vias 0 -> 1
- net D2: track 100.6 -> 185.8 mm
- net D1: track 93.3 -> 172.5 mm
- net Net-(C73-Pad1): track 0.00 -> 78.8 mm
- net Net-(C74-Pad1): track 0.00 -> 78.4 mm
- net CLK_IN: track 3.00 -> 80.0 mm, vias 0 -> 1
- net A10: track 156.2 -> 230.6 mm, vias 1 -> 3
- net D0: track 87.6 -> 161.8 mm
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
Commit message: Tracking
Connections:
- C18 pad 1: +5P -> +5VA
- J24 pad 13: +5P -> +5VA
- J4 pad 5: (no net) -> AUDIO
Routing:
- net A8: track 160.5 -> 344.6 mm, vias 1 -> 5
- net A9: track 161.8 -> 340.0 mm, vias 1 -> 5
- net A5: track 157.3 -> 318.9 mm, vias 1 -> 3
- net A6: track 151.6 -> 311.0 mm, vias 1 -> 3
- net A7: track 147.2 -> 302.0 mm, vias 1 -> 3
- net +5VA: track 1427.7 -> 1525.1 mm
- net PROCEED: track 8.30 -> 100.5 mm
- net A11: track 204.4 -> 291.4 mm, vias 3 -> 4
- net A12: track 220.5 -> 302.6 mm, vias 3 -> 4
- net READY: track 0.00 -> 79.6 mm, vias 0 -> 2
- net A10: track 230.6 -> 306.7 mm, vias 3 -> 4
- net MTR_CLR: track 0.00 -> 72.1 mm
- net A13: track 56.6 -> 128.4 mm, vias 0 -> 2
- net A4: track 163.2 -> 231.4 mm, vias 1 -> 2
- net D0: track 161.8 -> 225.3 mm, vias 0 -> 2
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
Commit message: Tracking
Parts:
- added FB7: Ferrite_Bead, Atari:L_Axial_L7.0mm_D3.3mm_P12.50mm_Horizontal_Fastron_MICC, F.Cu at (113.8, 45.5)
- moved C42 12.5 mm to (144.1, 115.0), turned to 180 degrees
- moved C24 0.63 mm to (65.0, 114.0)
- moved R11 0.54 mm to (64.1, 111.5)
Connections:
- M1 pad 1: COMPOSITE -> Net-(FB7-Pad1)
- M1 pad 4: MONO -> MONO_MOD
- Q3 pad 1: Net-(Q3-Pad1) -> MONO_MOD
- R204 pad 2: Net-(Q3-Pad1) -> MONO_MOD
- R37 pad 1: Net-(C47-Pad2) -> Net-(C46-Pad2)
- R37 pad 2: Net-(C46-Pad2) -> Net-(C47-Pad2)
- R53 pad 1: Net-(Q3-Pad1) -> MONO_MOD
Routing:
- net PB5: track 30.9 -> 256.7 mm, vias 0 -> 5
- net D1: track 230.5 -> 437.4 mm
- net EXTSEL: track 60.4 -> 263.1 mm, vias 1 -> 5
- net D0: track 225.3 -> 426.9 mm
- net D2: track 237.9 -> 431.0 mm
- net HALT: track 23.4 -> 194.5 mm, vias 1 -> 5
- net D3: track 234.7 -> 378.2 mm
- net CASINH: track 0.00 -> 138.3 mm, vias 0 -> 3
- net D4: track 202.1 -> 338.3 mm
- net AUDIO: track 0.00 -> 136.1 mm
- net O2: track 80.9 -> 211.7 mm, vias 1 -> 2
- net CHROMA: track 0.00 -> 124.6 mm, vias 0 -> 1
- net PB4: track 9.39 -> 128.7 mm, vias 0 -> 1
- net A13: track 128.4 -> 245.2 mm, vias 2 -> 7
- net PB3: track 13.3 -> 128.4 mm, vias 0 -> 1
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
Commit message: Tracking
Parts:
- moved C24 18.0 mm to (83.0, 114.0), turned to 180 degrees
- moved R11 12.5 mm to (64.0, 99.0), turned to 270 degrees
- moved C205 1.00 mm to (94.0, 60.4)
- moved C44 0.79 mm to (113.0, 66.7)
- moved R35 0.78 mm to (125.5, 69.2)
- moved Q1 0.74 mm to (104.9, 68.7)
- moved L13 0.60 mm to (90.6, 60.4)
Routing:
- net Net-(C48-Pad2): track 0.00 -> 147.8 mm, vias 0 -> 4
- net RD5: track 0.00 -> 125.3 mm, vias 0 -> 4
- net A1: track 250.8 -> 361.6 mm, vias 2 -> 4
- net A0: track 228.3 -> 337.2 mm, vias 1 -> 3
- net +5VA: track 1522.9 -> 1625.7 mm, vias 10 -> 14
- net GND: track 1205.3 -> 1302.5 mm, vias 4 -> 7
- net BELL: track 0.00 -> 96.9 mm
- net Net-(Q3-Pad2): track 14.2 -> 80.0 mm, vias 0 -> 1
- net Net-(Q3-Pad3): track 0.00 -> 44.4 mm
- net Net-(C19-Pad1): track 0.00 -> 25.3 mm
- net O1: track 0.00 -> 24.2 mm, vias 0 -> 1
- net Net-(C50-Pad1): track 0.00 -> 23.4 mm
- net Net-(D4-Pad2): track 0.00 -> 17.9 mm
- net Net-(R50-Pad2): track 0.00 -> 14.3 mm
- net Net-(C23-Pad1): track 0.00 -> 13.5 mm, vias 0 -> 1
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
Commit message: Tracking
Parts:
- removed C25: 100nF, Atari:C_Axial_L5.1mm_D2.5mm_P12.50mm_Horizontal
- added C22: 4,7uF, Capacitor_THT:CP_Radial_D8.0mm_P3.50mm, F.Cu at (124.8, 43.6)
- R18, R26: footprint Atari:R_Axial_DIN0207_L3.6mm_D2.2mm_P10.16mm_Horizontal -> Resistor_THT:R_Axial_DIN0207_L6.3mm_D2.5mm_P10.16mm_Horizontal
- moved R9 13.7 mm to (80.7, 76.0), turned to 180 degrees
- moved U34 3.94 mm to (61.3, 137.4)
- moved C103 3.64 mm to (62.5, 141.0)
- moved R23 3.64 mm to (62.5, 150.0)
- moved R24 3.64 mm to (62.5, 144.0)
- moved R25 3.64 mm to (62.5, 147.0)
- moved R110 3.00 mm to (63.5, 123.0)
- moved R111 3.00 mm to (63.5, 126.0)
- moved U3 1.78 mm to (101.9, 126.4)
- moved Q2 1.42 mm to (92.0, 115.4)
- moved C24 1.34 mm to (81.7, 113.6)
- moved R11 1.19 mm to (63.9, 97.8)
- moved R201 0.64 mm to (86.5, 118.6)
- moved C50 0.61 mm to (102.2, 103.0)
- moved C87 0.50 mm to (246.5, 63.0)
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Connections:
- C26 pad 1: +5P -> +5VA
- J4 pad 5: AUDIO -> EXTAUDIO
- R15 pad 1: +5P -> +5VA
- R72 pad 1: +5V -> +5VA
- U17 pad 30: O2 -> BO2
- U3 pad 20: +5P -> +5VA
Routing:
- net RST: track 55.9 -> 443.5 mm, vias 2 -> 8
- net MPD: track 0.00 -> 271.9 mm, vias 0 -> 4
- net +5VA: track 1625.7 -> 1893.6 mm, vias 14 -> 23
- net SIOAUDIO: track 0.00 -> 267.3 mm, vias 0 -> 5
- net REF: track 0.00 -> 263.0 mm, vias 0 -> 4
- net PB1: track 12.4 -> 245.2 mm, vias 1 -> 4
- net RD4: track 0.00 -> 227.5 mm, vias 0 -> 6
- net GND: track 1302.5 -> 1523.4 mm, vias 7 -> 8
- net S4: track 0.00 -> 210.3 mm, vias 0 -> 5
- net PB0: track 4.00 -> 205.9 mm, vias 0 -> 3
- net PB7: track 9.09 -> 196.8 mm, vias 0 -> 3
- net BO2: track 90.0 -> 275.8 mm, vias 1 -> 4
- net O2: track 211.7 -> 395.6 mm, vias 2 -> 4
- net IRQ: track 30.7 -> 208.3 mm, vias 0 -> 4
- net A15: track 100.7 -> 270.4 mm, vias 3 -> 6
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