File: Atari 130XE.kicad_pcb (KiCad board)
At the start: 2 copper layers, 324 x 204 mm, 325 parts, among them J1 SIO, J100 cond, J101 cond, J2 Video, J24 Cartridge, J4 Expansion, J5 Joystick_Port, J6 Joystick_Port, J7 Power, J8 Keyboard, M1 Modulator, Q1 2N3904, Q2 2N3904, Q3 2N3904, Q4 2N3906, Q6 2N3904, SW1 Switch_power_on, U1 LM358, U10 DRAM_4464, U11 DRAM_4464, U12 DRAM_4464, U17 GTIA, U18 74LS08, U19 LM555, U2 74LS138, U20 4050, U21 74LS74, U22 POKEY, U23 PIA, U24 CD4051B, U25 CD4051B, U3 MMU, U34 MMMU, U4 BASIC_ROM, U5 27C128, U6 Freddie, U7 Antic, U8 Sally, U9 DRAM_4464, Y1 Crystal, Y2 4,43 MHz

Commit message: Tracking
Parts:
- added J50: Conn_01x02, Connector_PinHeader_2.54mm:PinHeader_1x02_P2.54mm_Vertical, F.Cu at (81.6, 137.4)
- added J51: Conn_01x02, Connector_PinHeader_2.54mm:PinHeader_1x02_P2.54mm_Vertical, F.Cu at (81.6, 129.8)
- added R501: 3k, Atari:R_Axial_DIN0207_L3.6mm_D2.2mm_P10.16mm_Horizontal, F.Cu at (62.5, 153.0)
Connections:
- U23 pad 16: (no net) -> PB6
Routing:
- net GND: track 1523.4 -> 1533.6 mm
- net D4: track 336.1 -> 344.2 mm, vias 2 -> 3
- net A1: track 361.6 -> 369.6 mm, vias 4 -> 5
- net A2: track 253.0 -> 261.0 mm, vias 3 -> 4
- net A0: track 377.6 -> 385.6 mm, vias 4 -> 5
- net D5: track 196.3 -> 204.3 mm, vias 2 -> 3
- net D2: track 428.5 -> 436.4 mm, vias 2 -> 3
- net D1: track 435.4 -> 443.3 mm, vias 2 -> 3
- net CHROMA: track 125.0 -> 118.2 mm
- net +5VA: track 1893.6 -> 1896.6 mm
- net AUDIO: track 135.9 -> 134.4 mm
- net A13: track 293.3 -> 294.7 mm
- net CASINH: track 133.6 -> 134.7 mm
- net CAS: track 61.7 -> 62.5 mm

Commit message: Tracking
Connections:
- U17 pad 29: (no net) -> FO0
- U7 pad 35: (no net) -> FO0
Routing:
- net Net-(U18-Pad4): track 0.00 -> 134.3 mm, vias 0 -> 1
- net D4: track 344.2 -> 451.0 mm, vias 3 -> 6
- net D5: track 204.3 -> 306.4 mm, vias 3 -> 6
- net D2: track 436.4 -> 508.2 mm, vias 3 -> 5
- net D1: track 443.3 -> 513.6 mm, vias 3 -> 5
- net D0: track 435.6 -> 505.8 mm, vias 3 -> 5
- net O2: track 395.6 -> 456.2 mm, vias 4 -> 6
- net D3: track 375.9 -> 433.1 mm, vias 4 -> 5
- net FO0: track 0.00 -> 37.2 mm, vias 0 -> 1
- net +5VA: track 1896.6 -> 1930.9 mm, vias 23 -> 26
- net A12: track 359.2 -> 382.1 mm, vias 6 -> 7
- net REF: track 263.0 -> 262.0 mm
- net A10: track 306.3 -> 307.2 mm
- net PB5: track 256.9 -> 256.3 mm

Commit message: Tracking
Routing:
- net O0: track 0.00 -> 194.1 mm, vias 0 -> 4
- net A2: track 261.0 -> 441.8 mm, vias 4 -> 6
- net RW: track 126.5 -> 295.2 mm, vias 5 -> 8
- net A3: track 277.0 -> 434.7 mm, vias 5 -> 7
- net A1: track 369.6 -> 485.9 mm, vias 5 -> 6
- net A0: track 385.6 -> 498.8 mm, vias 5 -> 6
- net CCTL: track 37.8 -> 133.3 mm, vias 2 -> 4
- net D2: track 508.2 -> 546.7 mm
- net D1: track 513.6 -> 546.0 mm
- net D0: track 505.8 -> 532.7 mm
- net SIOAUDIO: track 267.3 -> 264.3 mm
- net +5VA: track 1930.9 -> 1928.5 mm
- net RD4: track 227.5 -> 225.6 mm
- net A10: track 307.2 -> 309.1 mm
- net Net-(R119-Pad2): track 34.5 -> 36.0 mm
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
Commit message: Tracking
Parts:
- moved C30 1.60 mm to (142.6, 89.0)
- moved Q1 0.30 mm to (104.9, 69.0)
Connections:
- U8 pad 5: GND -> (no net)
Routing:
- net RW: track 295.2 -> 486.9 mm, vias 8 -> 11
- net D7: track 258.1 -> 394.2 mm, vias 6 -> 7
- net Net-(U2-Pad4): track 0.00 -> 121.4 mm, vias 0 -> 1
- net Net-(R132-Pad2): track 49.6 -> 159.5 mm, vias 1 -> 2
- net GND: track 1533.6 -> 1640.2 mm
- net Net-(R133-Pad2): track 61.6 -> 165.0 mm, vias 0 -> 1
- net D5: track 306.4 -> 406.6 mm
- net D6: track 297.0 -> 394.3 mm
- net Net-(C206-Pad2): track 19.7 -> 96.9 mm, vias 0 -> 4
- net Net-(Q6-Pad3): track 8.58 -> 76.3 mm, vias 0 -> 3
- net RDY: track 10.1 -> 67.3 mm, vias 0 -> 1
- net NMI: track 36.4 -> 65.6 mm, vias 0 -> 1
- net E3: track 0.00 -> 18.1 mm, vias 0 -> 1
- net A4: track 338.4 -> 344.8 mm
- net A3: track 434.7 -> 439.5 mm
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- removed copper zone on F.Cu, net (none)

Commit message: Tracking
Parts:
- added J102: pin, Connector_PinHeader_2.00mm:PinHeader_1x01_P2.00mm_Vertical, F.Cu at (120.5, 66.7)
- moved C200 1.00 mm to (193.0, 154.3)
- moved R200 1.00 mm to (205.5, 157.3)
Routing:
- net PB6: track 0.00 -> 247.0 mm, vias 0 -> 5
- net D7: track 394.2 -> 447.3 mm
- net D6: track 394.3 -> 439.2 mm
- net D5: track 406.6 -> 446.5 mm
- net Net-(C44-Pad1): track 12.1 -> 19.6 mm
- net PB7: track 196.7 -> 194.8 mm
- net +5VA: track 1930.5 -> 1928.6 mm
- net Net-(C19-Pad1): track 121.0 -> 122.7 mm
- net GND: track 1640.2 -> 1638.6 mm
- net BASIC: track 90.6 -> 89.1 mm
- net D2: track 546.7 -> 545.5 mm
- net D1: track 546.0 -> 544.8 mm
- net D0: track 532.7 -> 531.4 mm
- net MPD: track 271.0 -> 272.1 mm
- net RW: track 486.9 -> 485.8 mm
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
Commit message: Gerber and Tracking
Parts:
- added J103: pin, Connector_PinHeader_2.00mm:PinHeader_1x01_P2.00mm_Vertical, F.Cu at (160.3, 99.4)
- added J104: pin, Connector_PinHeader_2.00mm:PinHeader_1x01_P2.00mm_Vertical, F.Cu at (189.9, 199.4)
- added J105: pin, Connector_PinHeader_2.00mm:PinHeader_1x01_P2.00mm_Vertical, F.Cu at (142.3, 189.9)
- added J106: pin, Connector_PinHeader_2.00mm:PinHeader_1x01_P2.00mm_Vertical, F.Cu at (147.8, 121.7)
- added J107: pin, Connector_PinHeader_2.00mm:PinHeader_1x01_P2.00mm_Vertical, F.Cu at (124.4, 150.8)
- added J108: pin, Connector_PinHeader_2.00mm:PinHeader_1x01_P2.00mm_Vertical, F.Cu at (343.4, 153.9)
- added J109: pin, Connector_PinHeader_2.00mm:PinHeader_1x01_P2.00mm_Vertical, F.Cu at (343.4, 150.9)
- added J110: pin, Connector_PinHeader_2.00mm:PinHeader_1x01_P2.00mm_Vertical, F.Cu at (343.4, 147.9)
- added J111: pin, Connector_PinHeader_2.00mm:PinHeader_1x01_P2.00mm_Vertical, F.Cu at (343.4, 144.9)
- C10, C2, C3: footprint Capacitor_THT:CP_Radial_D6.3mm_P2.50mm -> Capacitor_THT:CP_Axial_L11.0mm_D5.0mm_P18.00mm_Horizontal
- C79: footprint Capacitor_THT:CP_Radial_D5.0mm_P2.50mm -> Capacitor_THT:CP_Axial_L11.0mm_D5.0mm_P18.00mm_Horizontal
- moved C3 73.2 mm to (93.6, 63.2)
- moved C10 68.4 mm to (94.9, 79.2)
- moved C81 64.3 mm to (283.9, 87.9)
- moved R15 63.8 mm to (158.9, 174.9)
- moved U3 63.8 mm to (148.8, 169.7)
- moved R72 63.7 mm to (158.9, 177.7)
- moved H14 63.6 mm to (104.0, 69.9)
- moved R14 63.6 mm to (149.8, 173.1)
- moved C26 63.6 mm to (149.8, 179.0)
- moved R13 63.6 mm to (149.8, 176.0)
- moved L14 63.5 mm to (330.3, 216.9)
- moved R121 63.5 mm to (317.6, 110.6)
- moved C201 63.5 mm to (251.2, 182.6)
- moved C30 63.5 mm to (189.5, 131.9)
- moved C47 63.5 mm to (152.5, 91.9)
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Routing:
- net Net-(C1-Pad1): track 128.2 -> 111.7 mm
- net GND: track 1638.6 -> 1622.6 mm
- net +5VA: track 1928.6 -> 1918.2 mm, vias 26 -> 27
- net Net-(R140-Pad2): track 67.0 -> 58.4 mm, vias 1 -> 0
- net Net-(R144-Pad2): track 59.1 -> 50.9 mm, vias 1 -> 0
- net Net-(C111-Pad2): track 8.00 -> 15.5 mm
- net BELL: track 96.9 -> 104.4 mm
- net Net-(R142-Pad2): track 60.5 -> 53.1 mm
- net READY: track 79.3 -> 85.4 mm
- net Net-(R145-Pad2): track 44.5 -> 38.6 mm, vias 1 -> 0
- net Net-(C206-Pad2): track 96.9 -> 102.7 mm
- net Net-(C45-Pad1): track 16.6 -> 22.4 mm
- net +5C: track 147.7 -> 142.2 mm
- net Net-(R139-Pad2): track 72.1 -> 67.3 mm
- net Net-(R143-Pad2): track 56.1 -> 52.0 mm
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- added copper zone on F.Cu, net +5VA

Commit message: Trackimg
Parts:
- added J200: Diagnostic Signal, Connector_PinHeader_2.54mm:PinHeader_1x08_P2.54mm_Vertical, F.Cu at (69.1, 199.1)
- added J201: Diagnostic, Connector_PinHeader_2.54mm:PinHeader_1x04_P2.54mm_Vertical, F.Cu at (334.5, 112.6)
- added J202: Diag, Connector_PinHeader_2.54mm:PinHeader_1x04_P2.54mm_Vertical, F.Cu at (143.0, 62.1)
Routing:
- net RAS: track 104.7 -> 139.5 mm
- net O2: track 455.2 -> 487.2 mm, vias 6 -> 7
- net WRT: track 103.6 -> 134.9 mm
- net CAS: track 62.5 -> 90.2 mm
- net CASINH: track 134.6 -> 160.6 mm
- net OSC: track 128.9 -> 149.9 mm
- net EXTSEL: track 265.3 -> 285.3 mm
- net RW: track 485.8 -> 503.4 mm
- net BSC: track 64.0 -> 51.6 mm, vias 1 -> 0
- net GND: track 1622.6 -> 1618.0 mm
- net S4: track 209.0 -> 206.3 mm
- net COMPOSITE: track 30.3 -> 32.7 mm
- net DATA_OUT: track 102.1 -> 104.4 mm, vias 1 -> 0
- net A11: track 352.2 -> 350.2 mm
- net MONO: track 33.9 -> 35.7 mm
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Other:
- board text added: "74LS08"
- board text added: "74LS138"
- board text added: "74LS74"
- board text added: "ANTIC"
- board text added: "AUDIO"
- board text added: "BASIC"
- board text added: "CAS"
- board text added: "CASINH"
- board text added: "CD4050"
- board text added: "CD4051"
- board text added: "CHROMA"
- board text added: "Clk_in"
- board text added: "Clk_out"
- board text added: "Composite"
- board text added: "Data_in"
- board text added: "Data_out"
- board text added: "Diagnostic"
- board text added: "EXTSEL"
- board text added: "FREDDIE"
- board text added: "GTIA"
- board text added: "LM358"
- board text added: "LM555"
- board text added: "MONO"
- board text added: "O2"
- board text added: "OS"
- board text added: "OSC"
- board text added: "PIA"
- board text added: "POKEY"
- board text added: "RAS"
- board text added: "RW"
- board text added: "SALLY"
- board text added: "SDRAM4464"
- board text added: "SMMU"
- board text added: "WRT"

Commit message: Diagnostic
Parts:
- added J210: Diag, Connector_PinHeader_2.54mm:PinHeader_1x01_P2.54mm_Vertical, F.Cu at (158.0, 62.1)
- added J211: Diag, Connector_PinHeader_2.54mm:PinHeader_1x01_P2.54mm_Vertical, F.Cu at (327.3, 129.1)
- added J212: Diag, Connector_PinHeader_2.54mm:PinHeader_2x05_P2.54mm_Vertical, F.Cu at (242.2, 207.2)
- J200: value Diagnostic Signal -> Diag; footprint Connector_PinHeader_2.54mm:PinHeader_1x08_P2.54mm_Vertical -> Connector_PinHeader_2.54mm:PinHeader_1x10_P2.54mm_Vertical
- moved J200 0.26 mm to (68.8, 199.2)
Connections:
- J200 pad 2: EXTSEL -> REF
- J200 pad 3: RW -> EXTSEL
- J200 pad 4: OSC -> RW
- J200 pad 5: CASINH -> OSC
- J200 pad 6: CAS -> CASINH
- J200 pad 7: WRT -> CAS
- J200 pad 8: RAS -> WRT
- U2 pad 9: (no net) -> D6XX
- U8 pad 5: (no net) -> GND
Routing:
- net REF: track 262.3 -> 426.3 mm, vias 4 -> 7
- net A13: track 295.8 -> 294.4 mm
- net CASINH: track 160.6 -> 161.9 mm
- net EXTSEL: track 285.3 -> 286.6 mm
- net RAS: track 139.5 -> 140.8 mm
- net WRT: track 134.9 -> 136.1 mm
- net OSC: track 149.9 -> 151.2 mm
- net CAS: track 90.2 -> 91.5 mm
- net RW: track 503.4 -> 504.7 mm
Other:
- board text added: "GND"
- board text added: "REF"
