File: Ports.sch (KiCad schematic (older format))
At the start: 5 parts, among them J5 Joystick_Port, J6 Joystick_Port

Commit message: PIA and POKEY
Parts:
- added C93: 100nF, Atari:C_Axial_L5.1mm_D2.5mm_P12.50mm_Horizontal, symbol Device:C
- added C95: 10nF, Atari:C_Axial_L5.1mm_D2.5mm_P12.50mm_Horizontal, symbol Device:C
- added J1: SIO, Atari:SIO_Slot, symbol Atari:SIO_Port
- added J8: Keyboard, Connector_PinHeader_2.54mm:PinHeader_1x24_P2.54mm_Vertical, symbol Connector_Generic:Conn_01x24
- added R95: 1k, Atari:R_Axial_DIN0207_L3.6mm_D2.2mm_P10.16mm_Horizontal, symbol Device:R
Connections:
- net +5VA: now also C93.1, J8.1 (Pin_1), R95.2
- net GND: now also C93.2, C95.2, J1.4 (GND), J1.6 (GND), J8.3 (Pin_3)
- new net: C95.1, J8.2 (Pin_2), R95.1
- new net BSC: J8.20 (Pin_20)
- new net CLK_IN: J1.1 (CLK_IN)
- new net CLK_OUT: J1.2 (CLK_OUT)
- new net COMMAND: J1.7 (Command)
- new net DATA_IN: J1.3 (Data_In)
- new net DATA_OUT: J1.5 (Data_Out)
- new net IN0: J8.17 (Pin_17)
- new net IN1: J8.11 (Pin_11)
- new net IN2: J8.8 (Pin_8)
- new net IN3: J8.16 (Pin_16)
- new net IN4: J8.19 (Pin_19)
- new net IN5: J8.10 (Pin_10)
- new net IN6: J8.4 (Pin_4)
- new net IN7: J8.9 (Pin_9)
- new net INTRUPT: J1.13 (Intrupt)
- new net MTR_CLR: J1.8 (Mtr_Ctrl)
- new net OPTION: J8.23 (Pin_23)
- new net OUT0: J8.18 (Pin_18)
- new net OUT1: J8.13 (Pin_13)
- new net OUT2: J8.15 (Pin_15)
- new net OUT3: J8.5 (Pin_5)
- new net OUT4: J8.14 (Pin_14)
- new net OUT5: J8.6 (Pin_6)
- new net OUT6: J8.12 (Pin_12)
- new net OUT7: J8.7 (Pin_7)
- new net PROCEED: J1.9 (Proceed)
- new net READY: J1.10 (VCC)
- new net RESET: J8.24 (Pin_24)
- new net SELECT: J8.22 (Pin_22)
- new net SIOAUDIO: J1.11 (SIO_Audio)
- new net START: J8.21 (Pin_21)
Changed lines of the file:
@@
 	7025 2525 7025 2175
 Connection ~ 7475 2525
+$Comp
+L Atari:SIO_Port J1
+U 1 1 603D412B
+P 800 4175
+F 0 "J1" H 2628 4221 50  0000 L CNN
+F 1 "SIO" H 2628 4130 50  0000 L CNN
+F 2 "Atari:SIO_Slot" H 800 4175 50  0001 C CNN
+F 3 "" H 800 4175 50  0001 C CNN
+	1    800  4175
+	1    0    0    -1
+$EndComp
+Text GLabel 1850 4775 0    50   Input ~ 0
+CLK_IN
+Text GLabel 1850 4675 0    50   Input ~ 0
+CLK_OUT
+Text GLabel 1850 4575 0    50   Input ~ 0
+DATA_IN
+Text GLabel 1850 4375 0    50   Input ~ 0
+DATA_OUT
+Text GLabel 1850 4175 0    50   Input ~ 0
+COMMAND
+Text GLabel 1850 4075 0    50   Input ~ 0
+MTR_CLR
+Text GLabel 1850 3975 0    50   Input ~ 0
+PROCEED
+Text GLabel 1850 3775 0    50   Input ~ 0
+SIOAUDIO
+Text GLabel 1850 3575 0    50   Input ~ 0
+INTRUPT
+Wire Wire Line
+	1850 4275 1275 4275
+Wire Wire Line
+	1275 4275 1275 4475
+Wire Wire Line
+	1275 4475 1850 4475
+$Comp
+L power:GND #PWR0217
+U 1 1 603D6D5A
+P 1275 5000
+F 0 "#PWR0217" H 1275 4750 50  0001 C CNN
+F 1 "GND" H 1280 4827 50  0000 C CNN
+F 2 "" H 1275 5000 50  0001 C CNN
+F 3 "" H 1275 5000 50  0001 C CNN
+	1    1275 5000
+	1    0    0    -1
+$EndComp
+Wire Wire Line
+	1275 4475 1275 5000
+Connection ~ 1275 4475
+Text GLabel 1850 3875 0    50   Input ~ 0
+READY
+$Comp
+L Connector_Generic:Conn_01x24 J8
+U 1 1 603E550F
+P 5425 4275
+F 0 "J8" H 5505 4267 50  0000 L CNN
+F 1 "Keyboard" H 5505 4176 50  0000 L CNN
+F 2 "Connector_PinHeader_2.54mm:PinHeader_1x24_P2.54mm_Vertical" H 5425 4275 50  0001 C CNN
+F 3 "~" H 5425 4275 50  0001 C CNN
+	1    5425 4275
+	1    0    0    -1
+$EndComp
+Text GLabel 5225 5475 0    50   Input ~ 0
+RESET
+Text GLabel 5225 5375 0    50   Input ~ 0
+OPTION
+Text GLabel 5225 5275 0    50   Input ~ 0
+SELECT
+Text GLabel 5225 5175 0    50   Input ~ 0
+START
+Text GLabel 5225 5075 0    50   Input ~ 0
+BSC
+Text GLabel 5225 4975 0    50   Input ~ 0
+IN4
+Text GLabel 5225 4875 0    50   Input ~ 0
+OUT0
+Text GLabel 5225 4775 0    50   Input ~ 0
+IN0
+Text GLabel 5225 4675 0    50   Input ~ 0
+IN3
+Text GLabel 5225 4575 0    50   Input ~ 0
+OUT2
+Text GLabel 5225 4475 0    50   Input ~ 0
+OUT4
+Text GLabel 5225 4375 0    50   Input ~ 0
+OUT1
+Text GLabel 5225 4275 0    50   Input ~ 0
+OUT6
+Text GLabel 5225 4175 0    50   Input ~ 0
+IN1
+Text GLabel 5225 4075 0    50   Input ~ 0
+IN5
+Text GLabel 5225 3975 0    50   Input ~ 0
+IN7
+Text GLabel 5225 3875 0    50   Input ~ 0
+IN2
+Text GLabel 5225 3775 0    50   Input ~ 0
+OUT7
+Text GLabel 5225 3675 0    50   Input ~ 0
+OUT5
+Text GLabel 5225 3575 0    50   Input ~ 0
+OUT3
+Text GLabel 5225 3475 0    50   Input ~ 0
+IN6
+$Comp
+L power:GND #PWR0218
+U 1 1 603EA252
+P 4150 3525
+F 0 "#PWR0218" H 4150 3275 50  0001 C CNN
+F 1 "GND" H 4155 3352 50  0000 C CNN
+F 2 "" H 4150 3525 50  0001 C CNN
+F 3 "" H 4150 3525 50  0001 C CNN
+	1    4150 3525
+	1    0    0    -1
+$EndComp
+Wire Wire Line
+	4150 3375 4150 3525
+$Comp
+L Device:R R95
+U 1 1 603EACD2
+P 4550 3075
+F 0 "R95" V 4550 3075 50  0000 C CNN
+F 1 "1k" V 4500 2925 50  0000 C CNN
+F 2 "Atari:R_Axial_DIN0207_L3.6mm_D2.2mm_P10.16mm_Horizontal" V 4480 3075 50  0001 C CNN
+F 3 "~" H 4550 3075 50  0001 C CNN
+	1    4550 3075
+	0    1    1    0
+$EndComp
+$Comp
+L Device:C C93
+U 1 1 603EB979
+P 4150 3225
+F 0 "C93" H 4175 3300 50  0000 L CNN
+F 1 "100nF" H 4175 3150 50  0000 L CNN
+F 2 "Atari:C_Axial_L5.1mm_D2.5mm_P12.50mm_Horizontal" H 4188 3075 50  0001 C CNN
+F 3 "~" H 4150 3225 50  0001 C CNN
+	1    4150 3225
+	1    0    0    -1
+$EndComp
+Connection ~ 4150 3375
+Wire Wire Line
+	4150 3375 4900 3375
+$Comp
+L Device:C C95
+U 1 1 603ECF87
+P 4900 3225
+F 0 "C95" H 4750 3300 50  0000 L CNN
+F 1 "10nF" H 4700 3150 50  0000 L CNN
+F 2 "Atari:C_Axial_L5.1mm_D2.5mm_P12.50mm_Horizontal" H 4938 3075 50  0001 C CNN
+F 3 "~" H 4900 3225 50  0001 C CNN
+	1    4900 3225
+	1    0    0    -1
+$EndComp
+Connection ~ 4900 3375
+Wire Wire Line
+	4900 3375 5225 3375
+Wire Wire Line
+	4700 3075 4900 3075
+Wire Wire Line
+	4150 3075 4400 3075
+Wire Wire Line
+	5225 3275 5050 3275
+Wire Wire Line
+	5050 3275 5050 3075
+Wire Wire Line
+	5050 3075 4900 3075
+Connection ~ 4900 3075
+Wire Wire Line
+	5225 3175 5225 2875
+Wire Wire Line
+	5225 2875 4150 2875
+Wire Wire Line
+	4150 2875 4150 3075
+Connection ~ 4150 3075
+$Comp
+L power:+5VA #PWR0219
+U 1 1 603EF951
+P 4150 2750
+F 0 "#PWR0219" H 4150 2600 50  0001 C CNN
+F 1 "+5VA" H 4165 2923 50  0000 C CNN
+F 2 "" H 4150 2750 50  0001 C CNN
+F 3 "" H 4150 2750 50  0001 C CNN
+	1    4150 2750
+	1    0    0    -1
+$EndComp
+Wire Wire Line
+	4150 2750 4150 2875
+Connection ~ 4150 2875
 $EndSCHEMATC

Commit message: Pokey finish
Changed lines of the file:
@@
 	8075 2525 8075 2700
 Wire Wire Line
-	9175 2050 9175 3175
+	9175 2050 9175 2850
 Wire Wire Line
 	8075 3000 8075 3175
@@
 	4150 2750 4150 2875
 Connection ~ 4150 2875
+Text GLabel 9050 2850 0    50   Input ~ 0
+JOY_GND
+Wire Wire Line
+	9050 2850 9175 2850
+Connection ~ 9175 2850
+Wire Wire Line
+	9175 2850 9175 3175
 $EndSCHEMATC

Commit message: Schema finished
Parts:
- added C94: 10nF, Atari:C_Axial_L5.1mm_D2.5mm_P12.50mm_Horizontal, symbol Device:C
- added L25: 10uH, Atari:L_Axial_L7.0mm_D3.3mm_P12.50mm_Horizontal_Fastron_MICC, symbol Device:L
Connections:
- net +5P: now also L25.2; no longer C102.1, FB102.2
- net +5VA: now also C94.1
- net GND: now also C94.2
- net at FB102.1, J5.7 (VCC), J6.7 (VCC): now also C102.1
- new net: FB102.2, L25.1
Other:
- moved on the sheet: C102, C93, C95, FB102, FB12
Changed lines of the file:
@@
 L Device:Ferrite_Bead FB102
 U 1 1 602D4E49
-P 8675 2525
-F 0 "FB102" V 8401 2525 50  0000 C CNN
-F 1 "Ferrite_Bead" V 8492 2525 50  0000 C CNN
-F 2 "Atari:L_Axial_L7.0mm_D3.3mm_P12.50mm_Horizontal_Fastron_MICC" V 8605 2525 50  0001 C CNN
-F 3 "~" H 8675 2525 50  0001 C CNN
-	1    8675 2525
+P 8175 2525
+F 0 "FB102" V 8000 2500 50  0000 C CNN
+F 1 "Ferrite_Bead" V 8350 2500 50  0000 C CNN
+F 2 "Atari:L_Axial_L7.0mm_D3.3mm_P12.50mm_Horizontal_Fastron_MICC" V 8105 2525 50  0001 C CNN
+F 3 "~" H 8175 2525 50  0001 C CNN
+	1    8175 2525
 	0    1    1    0
 $EndComp
-Wire Wire Line
-	8825 2525 9300 2525
 Connection ~ 9300 2525
 Wire Wire Line
@@
 L Device:C C102
 U 1 1 602D5898
-P 8075 2850
-F 0 "C102" H 8190 2896 50  0000 L CNN
-F 1 "1nF" H 8190 2805 50  0000 L CNN
-F 2 "Atari:C_Axial_L5.1mm_D2.5mm_P12.50mm_Horizontal" H 8113 2700 50  0001 C CNN
-F 3 "~" H 8075 2850 50  0001 C CNN
-	1    8075 2850
-	1    0    0    -1
-$EndComp
-Wire Wire Line
-	8525 2525 8075 2525
-Wire Wire Line
-	8075 2525 8075 2700
-Wire Wire Line
-	9175 2050 9175 2850
-Wire Wire Line
-	8075 3000 8075 3175
-Wire Wire Line
-	8075 3175 9175 3175
+P 8625 2850
+F 0 "C102" H 8740 2896 50  0000 L CNN
+F 1 "1nF" H 8740 2805 50  0000 L CNN
+F 2 "Atari:C_Axial_L5.1mm_D2.5mm_P12.50mm_Horizontal" H 8663 2700 50  0001 C CNN
+F 3 "~" H 8625 2850 50  0001 C CNN
+	1    8625 2850
+	1    0    0    -1
+$EndComp
+Wire Wire Line
+	8075 3175 8625 3175
 Connection ~ 9175 3175
 Wire Wire Line
@@
 Wire Wire Line
 	8075 3425 8075 3175
-Connection ~ 8075 3175
 $Comp
 L Device:Ferrite_Bead FB12
 U 1 1 602D6C5C
-P 7475 2325
-F 0 "FB12" H 7338 2279 50  0000 R CNN
-F 1 "Ferrite_Bead" H 7338 2370 50  0000 R CNN
-F 2 "Atari:L_Axial_L7.0mm_D3.3mm_P12.50mm_Horizontal_Fastron_MICC" V 7405 2325 50  0001 C CNN
-F 3 "~" H 7475 2325 50  0001 C CNN
-	1    7475 2325
+P 7050 2325
+F 0 "FB12" H 7275 2175 50  0000 R CNN
+F 1 "Ferrite_Bead" V 6875 2225 50  0000 R CNN
+F 2 "Atari:L_Axial_L7.0mm_D3.3mm_P12.50mm_Horizontal_Fastron_MICC" V 6980 2325 50  0001 C CNN
+F 3 "~" H 7050 2325 50  0001 C CNN
+	1    7050 2325
 	-1   0    0    1
 $EndComp
 Wire Wire Line
-	7475 2475 7475 2525
-Wire Wire Line
-	7475 2525 8075 2525
-Connection ~ 8075 2525
+	7050 2475 7050 2525
 $Comp
 L power:+5VA #PWR0195
 U 1 1 602D7D9F
-P 7475 2175
-F 0 "#PWR0195" H 7475 2025 50  0001 C CNN
-F 1 "+5VA" H 7490 2348 50  0000 C CNN
-F 2 "" H 7475 2175 50  0001 C CNN
-F 3 "" H 7475 2175 50  0001 C CNN
-	1    7475 2175
+P 7050 2175
+F 0 "#PWR0195" H 7050 2025 50  0001 C CNN
+F 1 "+5VA" H 7065 2348 50  0000 C CNN
+F 2 "" H 7050 2175 50  0001 C CNN
+F 3 "" H 7050 2175 50  0001 C CNN
+	1    7050 2175
 	1    0    0    -1
 $EndComp
@@
 L power:+5P #PWR0196
 U 1 1 602D9976
-P 7025 2175
-F 0 "#PWR0196" H 7025 2025 50  0001 C CNN
-F 1 "+5P" H 7040 2348 50  0000 C CNN
-F 2 "" H 7025 2175 50  0001 C CNN
-F 3 "" H 7025 2175 50  0001 C CNN
-	1    7025 2175
-	1    0    0    -1
-$EndComp
-Wire Wire Line
-	7475 2525 7025 2525
-Wire Wire Line
-	7025 2525 7025 2175
-Connection ~ 7475 2525
+P 7375 2175
+F 0 "#PWR0196" H 7375 2025 50  0001 C CNN
+F 1 "+5P" H 7390 2348 50  0000 C CNN
+F 2 "" H 7375 2175 50  0001 C CNN
+F 3 "" H 7375 2175 50  0001 C CNN
+	1    7375 2175
+	1    0    0    -1
+$EndComp
 $Comp
 L Atari:SIO_Port J1
@@
 L Device:C C93
 U 1 1 603EB979
-P 4150 3225
-F 0 "C93" H 4175 3300 50  0000 L CNN
-F 1 "100nF" H 4175 3150 50  0000 L CNN
-F 2 "Atari:C_Axial_L5.1mm_D2.5mm_P12.50mm_Horizontal" H 4188 3075 50  0001 C CNN
-F 3 "~" H 4150 3225 50  0001 C CNN
-	1    4150 3225
+P 3675 3225
+F 0 "C93" H 3700 3300 50  0000 L CNN
+F 1 "100nF" H 3700 3150 50  0000 L CNN
+F 2 "Atari:C_Axial_L5.1mm_D2.5mm_P12.50mm_Horizontal" H 3713 3075 50  0001 C CNN
+F 3 "~" H 3675 3225 50  0001 C CNN
+	1    3675 3225
 	1    0    0    -1
 $EndComp
 Connection ~ 4150 3375
-Wire Wire Line
-	4150 3375 4900 3375
 $Comp
 L Device:C C95
 U 1 1 603ECF87
-P 4900 3225
-F 0 "C95" H 4750 3300 50  0000 L CNN
-F 1 "10nF" H 4700 3150 50  0000 L CNN
-F 2 "Atari:C_Axial_L5.1mm_D2.5mm_P12.50mm_Horizontal" H 4938 3075 50  0001 C CNN
-F 3 "~" H 4900 3225 50  0001 C CNN
-	1    4900 3225
-	1    0    0    -1
-$EndComp
-Connection ~ 4900 3375
-Wire Wire Line
-	4900 3375 5225 3375
-Wire Wire Line
-	4700 3075 4900 3075
+P 5050 3225
+F 0 "C95" H 4900 3300 50  0000 L CNN
+F 1 "10nF" H 4850 3150 50  0000 L CNN
+F 2 "Atari:C_Axial_L5.1mm_D2.5mm_P12.50mm_Horizontal" H 5088 3075 50  0001 C CNN
+F 3 "~" H 5050 3225 50  0001 C CNN
+	1    5050 3225
+	1    0    0    -1
+$EndComp
 Wire Wire Line
 	4150 3075 4400 3075
-Wire Wire Line
-	5225 3275 5050 3275
-Wire Wire Line
-	5050 3275 5050 3075
-Wire Wire Line
-	5050 3075 4900 3075
-Connection ~ 4900 3075
 Wire Wire Line
 	5225 3175 5225 2875
@@
 	4150 2750 4150 2875
 Connection ~ 4150 2875
-Text GLabel 9050 2850 0    50   Input ~ 0
-JOY_GND
-Wire Wire Line
-	9050 2850 9175 2850
-Connection ~ 9175 2850
-Wire Wire Line
-	9175 2850 9175 3175
+$Comp
+L Device:L L25
+U 1 1 602F3A65
+P 7550 2525
+F 0 "L25" V 7369 2525 50  0000 C CNN
+F 1 "10uH" V 7460 2525 50  0000 C CNN
+F 2 "Atari:L_Axial_L7.0mm_D3.3mm_P12.50mm_Horizontal_Fastron_MICC" H 7550 2525 50  0001 C CNN
+F 3 "~" H 7550 2525 50  0001 C CNN
+	1    7550 2525
+	0    1    1    0
+$EndComp
+Wire Wire Line
+	9175 2050 9175 3175
+Wire Wire Line
+	8625 2700 8625 2525
+Wire Wire Line
+	8625 2525 9300 2525
+Wire Wire Line
+	8625 3000 8625 3175
+Connection ~ 8625 3175
+Wire Wire Line
+	8625 3175 9175 3175
+Wire Wire Line
+	8325 2525 8625 2525
+Connection ~ 8625 2525
+Wire Wire Line
+	7050 2525 7375 2525
+Wire Wire Line
+	7700 2525 8025 2525
+Wire Wire Line
+	7375 2175 7375 2525
+Connection ~ 7375 2525
+Wire Wire Line
+	7375 2525 7400 2525
+Connection ~ 5050 3375
+Wire Wire Line
+	5050 3375 5225 3375
+Wire Wire Line
+	5050 3075 5175 3075
+Wire Wire Line
+	5175 3075 5175 3275
+Wire Wire Line
+	5175 3275 5225 3275
+Connection ~ 5050 3075
+$Comp
+L Device:C C94
+U 1 1 60336678
+P 4150 3225
+F 0 "C94" H 4000 3300 50  0000 L CNN
+F 1 "10nF" H 3950 3150 50  0000 L CNN
+F 2 "Atari:C_Axial_L5.1mm_D2.5mm_P12.50mm_Horizontal" H 4188 3075 50  0001 C CNN
+F 3 "~" H 4150 3225 50  0001 C CNN
+	1    4150 3225
+	1    0    0    -1
+$EndComp
+Wire Wire Line
+	4700 3075 5050 3075
+Wire Wire Line
+	4150 3375 5050 3375
+Wire Wire Line
+	3675 3075 4150 3075
+Wire Wire Line
+	3675 3375 4150 3375
 $EndSCHEMATC
