File: Power.sch (KiCad schematic (older format))
At the start: 2 parts, among them J7 Power, SW1 Switch_power_on

Commit message: Memory and Freddie
Parts:
- added C1: 470uF, Capacitor_THT:CP_Radial_D8.0mm_P3.80mm, symbol Device:CP
- added C10, C2, C3: 22uF, Capacitor_THT:CP_Radial_D6.3mm_P2.50mm, symbol Device:CP
- added C11, C7: 10nF, Atari:C_Axial_L5.1mm_D2.5mm_P12.50mm_Horizontal, symbol Device:C
- added C12, C14, C15, C5, C6, C8, C9: 1nF, Atari:C_Axial_L5.1mm_D2.5mm_P12.50mm_Horizontal, symbol Device:C
- added C13, C205, C4: 100nF, Atari:C_Axial_L5.1mm_D2.5mm_P12.50mm_Horizontal, symbol Device:C
- added FB1, FB2, FB3: Ferrite_Bead, Atari:L_Axial_L7.0mm_D3.3mm_P12.50mm_Horizontal_Fastron_MICC, symbol Device:Ferrite_Bead
- added L13: 820uH, Atari:L_Axial_L7.0mm_D3.3mm_P12.50mm_Horizontal_Fastron_MICC, symbol Device:L
Connections:
- net GND: now also C1.2, C10.2, C11.2, C12.2, C13.2, C14.2, C15.2, C2.2, C205.2, C3.2, C4.2, C5.2, C6.2, C7.2, C8.2, C9.2
- net at SW1.2 (Out): now also C1.1, C2.1, C3.1, C4.1, C5.1, C6.1, C7.1, FB1.2, FB2.2, FB3.2
- new net: C205.1, L13.1
- new net +5C: C10.1, C13.1, C15.1, FB3.1, L13.2
- new net +5V: C12.1, C14.1, C9.1, FB2.1
- new net +5VA: C11.1, C8.1, FB1.1

Commit message: MMU, Joy, Cart and Video
Connections:
- net RF_VCC: now reaches C205.1, L13.1
Changed lines of the file:
@@
 $Descr A4 11693 8268
 encoding utf-8
-Sheet 3 14
+Sheet 3 15
 Title ""
 Date ""
@@
 Wire Wire Line
 	7775 4150 7775 4225
+Text GLabel 8275 3850 2    50   Input ~ 0
+RF_VCC
+Wire Wire Line
+	7775 3850 8275 3850
+Connection ~ 7775 3850
+$Comp
+L power:+5P #PWR0183
+U 1 1 602DB6E0
+P 3625 6400
+F 0 "#PWR0183" H 3625 6250 50  0001 C CNN
+F 1 "+5P" H 3640 6573 50  0000 C CNN
+F 2 "" H 3625 6400 50  0001 C CNN
+F 3 "" H 3625 6400 50  0001 C CNN
+	1    3625 6400
+	1    0    0    -1
+$EndComp
+$Comp
+L power:PWR_FLAG #FLG0105
+U 1 1 602DBADD
+P 3625 6700
+F 0 "#FLG0105" H 3625 6775 50  0001 C CNN
+F 1 "PWR_FLAG" H 3625 6873 50  0000 C CNN
+F 2 "" H 3625 6700 50  0001 C CNN
+F 3 "~" H 3625 6700 50  0001 C CNN
+	1    3625 6700
+	-1   0    0    1
+$EndComp
+Wire Wire Line
+	3625 6400 3625 6700
 $EndSCHEMATC

Commit message: Gerber and Tracking
Parts:
- C10, C2, C3: footprint Capacitor_THT:CP_Radial_D6.3mm_P2.50mm -> Capacitor_THT:CP_Axial_L11.0mm_D5.0mm_P18.00mm_Horizontal
Changed lines of the file:
@@
 F 0 "C3" H 3918 3046 50  0000 L CNN
 F 1 "22uF" H 3918 2955 50  0000 L CNN
-F 2 "Capacitor_THT:CP_Radial_D6.3mm_P2.50mm" H 3838 2850 50  0001 C CNN
+F 2 "Capacitor_THT:CP_Axial_L11.0mm_D5.0mm_P18.00mm_Horizontal" H 3838 2850 50  0001 C CNN
 F 3 "~" H 3800 3000 50  0001 C CNN
 	1    3800 3000
@@
 F 0 "C2" H 4318 1871 50  0000 L CNN
 F 1 "22uF" H 4318 1780 50  0000 L CNN
-F 2 "Capacitor_THT:CP_Radial_D6.3mm_P2.50mm" H 4238 1675 50  0001 C CNN
+F 2 "Capacitor_THT:CP_Axial_L11.0mm_D5.0mm_P18.00mm_Horizontal" H 4238 1675 50  0001 C CNN
 F 3 "~" H 4200 1825 50  0001 C CNN
 	1    4200 1825
@@
 F 0 "C10" H 5993 4046 50  0000 L CNN
 F 1 "22uF" H 5993 3955 50  0000 L CNN
-F 2 "Capacitor_THT:CP_Radial_D6.3mm_P2.50mm" H 5913 3850 50  0001 C CNN
+F 2 "Capacitor_THT:CP_Axial_L11.0mm_D5.0mm_P18.00mm_Horizontal" H 5913 3850 50  0001 C CNN
 F 3 "~" H 5875 4000 50  0001 C CNN
 	1    5875 4000
