File: GTIA.sch (KiCad schematic (older format))
At the start: 72 parts, among them J2 Video, Q1 2N3904, Q2 2N3904, Q3 2N3904, Q6 2N3904, U17 GTIA, U18 74LS08, U20 4050, U21 74LS74, Y2 4,43 MHz

Commit message: Tracking
Parts:
- added J102: pin, Connector_PinHeader_2.00mm:PinHeader_1x01_P2.00mm_Vertical, symbol Connector_Generic:Conn_01x01
Connections:
- net at C44.1, Q1.2 (B), R35.2: now also J102.1 (Pin_1)
Changed lines of the file:
@@
 	1    0    0    -1
 $EndComp
+$Comp
+L Connector_Generic:Conn_01x01 J102
+U 1 1 6037C604
+P 800 6575
+F 0 "J102" H 950 6475 50  0000 C CNN
+F 1 "pin" H 718 6441 50  0000 C CNN
+F 2 "Connector_PinHeader_2.00mm:PinHeader_1x01_P2.00mm_Vertical" H 800 6575 50  0001 C CNN
+F 3 "~" H 800 6575 50  0001 C CNN
+	1    800  6575
+	-1   0    0    1
+$EndComp
+Wire Wire Line
+	1000 6575 1200 6575
+Wire Wire Line
+	1200 6575 1200 6200
 $EndSCHEMATC

Commit message: Gerber and Tracking
Parts:
- added J103, J104, J105: pin, Connector_PinHeader_2.00mm:PinHeader_1x01_P2.00mm_Vertical, symbol Connector_Generic:Conn_01x01
Connections:
- net at C206.2, L37.1, U17.28 (OSC)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: now also J104.1 (Pin_1)
- net at C45.1, D2.1 (K), D3.2 (A): now also J103.1 (Pin_1)
- net at C111.2, C61.2, L8.2: now also J105.1 (Pin_1)
Changed lines of the file:
@@
 Wire Wire Line
 	1200 6575 1200 6200
+$Comp
+L Connector_Generic:Conn_01x01 J103
+U 1 1 603DC950
+P 2375 6400
+F 0 "J103" H 2525 6300 50  0000 C CNN
+F 1 "pin" H 2293 6266 50  0000 C CNN
+F 2 "Connector_PinHeader_2.00mm:PinHeader_1x01_P2.00mm_Vertical" H 2375 6400 50  0001 C CNN
+F 3 "~" H 2375 6400 50  0001 C CNN
+	1    2375 6400
+	0    1    1    0
+$EndComp
+Wire Wire Line
+	2375 6200 2375 6000
+$Comp
+L Connector_Generic:Conn_01x01 J104
+U 1 1 603FEA4A
+P 5125 6250
+F 0 "J104" H 5275 6150 50  0000 C CNN
+F 1 "pin" H 5043 6116 50  0000 C CNN
+F 2 "Connector_PinHeader_2.00mm:PinHeader_1x01_P2.00mm_Vertical" H 5125 6250 50  0001 C CNN
+F 3 "~" H 5125 6250 50  0001 C CNN
+	1    5125 6250
+	-1   0    0    1
+$EndComp
+Wire Wire Line
+	5325 6250 5425 6250
+Connection ~ 5425 6250
+$Comp
+L Connector_Generic:Conn_01x01 J105
+U 1 1 6041A994
+P 6150 7550
+F 0 "J105" H 6300 7450 50  0000 C CNN
+F 1 "pin" H 6068 7416 50  0000 C CNN
+F 2 "Connector_PinHeader_2.00mm:PinHeader_1x01_P2.00mm_Vertical" H 6150 7550 50  0001 C CNN
+F 3 "~" H 6150 7550 50  0001 C CNN
+	1    6150 7550
+	0    1    1    0
+$EndComp
+Wire Wire Line
+	6150 7350 6150 7125
+Connection ~ 6150 7125
 $EndSCHEMATC

Commit message: Trackimg
Parts:
- added J202: Diag, Connector_PinHeader_2.54mm:PinHeader_1x04_P2.54mm_Vertical, symbol Connector_Generic:Conn_01x04
Connections:
- net AUDIO: now also J202.4 (Pin_4)
- net CHROMA: now also J202.3 (Pin_3)
- net COMPOSITE: now also J202.1 (Pin_1)
- net MONO: now also J202.2 (Pin_2)
Changed lines of the file:
@@
 	6150 7350 6150 7125
 Connection ~ 6150 7125
+Text GLabel 2650 7200 0    50   Input ~ 0
+MONO
+Text GLabel 2650 7100 0    50   Input ~ 0
+COMPOSITE
+Text GLabel 2650 7300 0    50   Input ~ 0
+CHROMA
+Text GLabel 2650 7400 0    50   Input ~ 0
+AUDIO
+$Comp
+L Connector_Generic:Conn_01x04 J202
+U 1 1 6046696D
+P 2850 7200
+F 0 "J202" H 2930 7192 50  0000 L CNN
+F 1 "Diag" H 2930 7101 50  0000 L CNN
+F 2 "Connector_PinHeader_2.54mm:PinHeader_1x04_P2.54mm_Vertical" H 2850 7200 50  0001 C CNN
+F 3 "~" H 2850 7200 50  0001 C CNN
+	1    2850 7200
+	1    0    0    -1
+$EndComp
 $EndSCHEMATC

Commit message: Diagnostic
Parts:
- added J210: Diag, Connector_PinHeader_2.54mm:PinHeader_1x01_P2.54mm_Vertical, symbol Connector_Generic:Conn_01x01
Connections:
- net GND: now also J210.1 (Pin_1)
Changed lines of the file:
@@
 	1    0    0    -1
 $EndComp
+$Comp
+L power:GND #PWR0253
+U 1 1 60456DB7
+P 3350 7500
+F 0 "#PWR0253" H 3350 7250 50  0001 C CNN
+F 1 "GND" H 3355 7327 50  0000 C CNN
+F 2 "" H 3350 7500 50  0001 C CNN
+F 3 "" H 3350 7500 50  0001 C CNN
+	1    3350 7500
+	1    0    0    -1
+$EndComp
+$Comp
+L Connector_Generic:Conn_01x01 J210
+U 1 1 6046AFBB
+P 3550 7300
+F 0 "J210" H 3630 7342 50  0000 L CNN
+F 1 "Diag" H 3630 7251 50  0000 L CNN
+F 2 "Connector_PinHeader_2.54mm:PinHeader_1x01_P2.54mm_Vertical" H 3550 7300 50  0001 C CNN
+F 3 "~" H 3550 7300 50  0001 C CNN
+	1    3550 7300
+	1    0    0    -1
+$EndComp
+Wire Wire Line
+	3350 7300 3350 7500
 $EndSCHEMATC
