File: MMU.sch (KiCad schematic (older format))
At the start: 0 parts

Commit message: MMU, Joy, Cart and Video
Parts:
- added C25, C26: 100nF, Atari:C_Axial_L5.1mm_D2.5mm_P12.50mm_Horizontal, symbol Device:C
- added R12, R15: 3k, Atari:R_Axial_DIN0207_L3.6mm_D2.2mm_P10.16mm_Horizontal, symbol Device:R
- added R13, R14: 1k, Atari:R_Axial_DIN0207_L3.6mm_D2.2mm_P10.16mm_Horizontal, symbol Device:R
- added U18: 74LS08, Package_DIP:DIP-14_W7.62mm_Socket, symbol 74xx:74LS08
- added U2: 74LS138, Package_DIP:DIP-16_W7.62mm_Socket, symbol 74xx:74LS138
- added U3: MMU, Package_DIP:DIP-20_W7.62mm_Socket, symbol Atari:MMU
Connections:
- new net: U18.10, U18.9, U2.15 (O0)
- new net: U2.4 (E1), U3.17 (~IO)
- new net +5P: C25.1, C26.1, R12.1, R15.1, U2.16 (VCC), U3.20 (VCC)
- new net A10: U2.3 (A2)
- new net A11: U3.1 (A11)
- new net A12: U3.2 (A12)
- new net A13: U3.3 (A13)
- new net A14: U3.4 (A14)
- new net A15: U3.5 (A15)
- new net A8: U2.1 (A0)
- new net A9: U2.2 (A1)
- new net BASIC: U3.13 (~BASIC)
- new net CASINH: U3.16 (~CI)
- new net CCTL: U2.10 (O5)
- new net D1XX: U2.14 (O1)
- new net E3: R12.2, U2.6 (E3)
- new net GND: C25.2, C26.2, R13.2, R14.2, U2.5 (E2), U2.8 (GND), U3.10 (VSS)
- new net GTIA: U18.8
- new net MPD: R15.2, U3.14 (~MPD)
- new net OS: U3.15 (~OS)
- new net PB0: U3.9 (REN)
- new net PB1: U3.18 (~BE)
- new net PB7: U3.6 (~MAP)
- new net PIA: U2.12 (O3)
- new net POKEY: U2.13 (O2)
- new net RD4: R14.1, U3.7 (RD4)
- new net RD5: R13.1, U3.8 (RD5)
- new net REF: U3.11 (~REF)
- new net S4: U3.19 (~S4)
- new net S5: U3.12 (~S5)
- no-connect marks 0 -> 3

Commit message: Schema finished
Connections:
- net +5P: no longer C25.1, R12.1, U2.16 (VCC)
- new net +5VA: C25.1, R12.1, U2.16 (VCC)
Changed lines of the file:
@@
 Text GLabel 1775 2275 3    50   Input ~ 0
 E3
-$Comp
-L power:+5P #PWR0189
-U 1 1 602E9089
-P 1775 1750
-F 0 "#PWR0189" H 1775 1600 50  0001 C CNN
-F 1 "+5P" H 1790 1923 50  0000 C CNN
-F 2 "" H 1775 1750 50  0001 C CNN
-F 3 "" H 1775 1750 50  0001 C CNN
-	1    1775 1750
-	1    0    0    -1
-$EndComp
 Wire Wire Line
 	1775 2175 1775 2275
@@
 Wire Wire Line
 	2600 2175 2600 2275
-$Comp
-L power:+5P #PWR0192
-U 1 1 602F3B32
-P 5375 1575
-F 0 "#PWR0192" H 5375 1425 50  0001 C CNN
-F 1 "+5P" H 5390 1748 50  0000 C CNN
-F 2 "" H 5375 1575 50  0001 C CNN
-F 3 "" H 5375 1575 50  0001 C CNN
-	1    5375 1575
-	1    0    0    -1
-$EndComp
 Wire Wire Line
 	5375 1575 5375 1750
@@
 	5375 3050 5375 3200
 Connection ~ 5375 3050
+$Comp
+L power:+5VA #PWR0189
+U 1 1 60310513
+P 1775 1750
+F 0 "#PWR0189" H 1775 1600 50  0001 C CNN
+F 1 "+5VA" H 1790 1923 50  0000 C CNN
+F 2 "" H 1775 1750 50  0001 C CNN
+F 3 "" H 1775 1750 50  0001 C CNN
+	1    1775 1750
+	1    0    0    -1
+$EndComp
+$Comp
+L power:+5VA #PWR?
+U 1 1 60350D58
+P 5375 1575
+F 0 "#PWR?" H 5375 1425 50  0001 C CNN
+F 1 "+5VA" H 5390 1748 50  0000 C CNN
+F 2 "" H 5375 1575 50  0001 C CNN
+F 3 "" H 5375 1575 50  0001 C CNN
+	1    5375 1575
+	1    0    0    -1
+$EndComp
 $EndSCHEMATC

Commit message: Tracking
Parts:
- removed C25: 100nF, Atari:C_Axial_L5.1mm_D2.5mm_P12.50mm_Horizontal, symbol Device:C
Connections:
- net +5P is gone; now on net +5VA: C26.1, R15.1, U3.20 (VCC)
Changed lines of the file:
@@
 MPD
-$Comp
-L power:+5P #PWR0184
-U 1 1 602E291A
-P 1475 1750
-F 0 "#PWR0184" H 1475 1600 50  0001 C CNN
-F 1 "+5P" H 1490 1923 50  0000 C CNN
-F 2 "" H 1475 1750 50  0001 C CNN
-F 3 "" H 1475 1750 50  0001 C CNN
-	1    1475 1750
-	1    0    0    -1
-$EndComp
 $Comp
 L Device:R R15
@@
 	4325 5500 4325 5600
 Connection ~ 4325 5500
-$Comp
-L power:+5P #PWR0187
-U 1 1 602E6C38
-P 4325 5075
-F 0 "#PWR0187" H 4325 4925 50  0001 C CNN
-F 1 "+5P" H 4340 5248 50  0000 C CNN
-F 2 "" H 4325 5075 50  0001 C CNN
-F 3 "" H 4325 5075 50  0001 C CNN
-	1    4325 5075
-	1    0    0    -1
-$EndComp
 Wire Wire Line
 	4325 5075 4325 5200
@@
 NoConn ~ 5875 2750
 $Comp
-L Device:C C25
-U 1 1 602EB98F
-P 6725 2350
-F 0 "C25" H 6840 2396 50  0000 L CNN
-F 1 "100nF" H 6840 2305 50  0000 L CNN
-F 2 "Atari:C_Axial_L5.1mm_D2.5mm_P12.50mm_Horizontal" H 6763 2200 50  0001 C CNN
-F 3 "~" H 6725 2350 50  0001 C CNN
-	1    6725 2350
-	1    0    0    -1
-$EndComp
-Wire Wire Line
-	5375 1750 6725 1750
-Wire Wire Line
-	6725 1750 6725 2200
-Wire Wire Line
-	5375 3050 6725 3050
-Wire Wire Line
-	6725 3050 6725 2500
-$Comp
 L 74xx:74LS08 U18
 U 3 1 602ED5C7
@@
 Wire Wire Line
 	5375 1575 5375 1750
-Connection ~ 5375 1750
 $Comp
 L power:GND #PWR0193
@@
 Wire Wire Line
 	5375 3050 5375 3200
-Connection ~ 5375 3050
 $Comp
 L power:+5VA #PWR0189
@@
 	1    0    0    -1
 $EndComp
+$Comp
+L power:+5VA #PWR0184
+U 1 1 60367244
+P 4325 5075
+F 0 "#PWR0184" H 4325 4925 50  0001 C CNN
+F 1 "+5VA" H 4340 5248 50  0000 C CNN
+F 2 "" H 4325 5075 50  0001 C CNN
+F 3 "" H 4325 5075 50  0001 C CNN
+	1    4325 5075
+	1    0    0    -1
+$EndComp
+$Comp
+L power:+5VA #PWR0187
+U 1 1 6036DC67
+P 1475 1750
+F 0 "#PWR0187" H 1475 1600 50  0001 C CNN
+F 1 "+5VA" H 1490 1923 50  0000 C CNN
+F 2 "" H 1475 1750 50  0001 C CNN
+F 3 "" H 1475 1750 50  0001 C CNN
+	1    1475 1750
+	1    0    0    -1
+$EndComp

Commit message: Diagnostic
Connections:
- net D4XX: now reaches U2.11 (O4)
- net D7XX: now reaches U2.7 (O7)
- net D6XX: now reaches U2.9 (O6)
- no-connect marks 3 -> 0
Changed lines of the file:
@@
 Text GLabel 5875 2250 2    50   Input ~ 0
 POKEY
-NoConn ~ 5875 2450
-NoConn ~ 5875 2650
-NoConn ~ 5875 2750
 $Comp
 L 74xx:74LS08 U18
@@
 	1    0    0    -1
 $EndComp
+Text GLabel 5875 2650 2    50   Input ~ 0
+D6XX
+Text GLabel 5875 2450 2    50   Input ~ 0
+D4XX
+Text GLabel 5875 2750 2    50   Input ~ 0
+D7XX
 $EndSCHEMATC
